File: schematics/DykoDAC_Output.sch (KiCad schematic (older format))
At the start: 41 parts

Commit message: changed filter values, and cap in osscilator power supply.
Parts:
- C? (x4): value 2n2 -> 1n
- C? (x4): value 6n8 -> 3n3
- R? (x4): value 1k2 -> 1k5
- R? (x8): value 1k2 -> 820
Changed lines of the file:
@@
 P 3350 4000
 F 0 "C?" H 3465 4046 50  0000 L CNN
-F 1 "2n2" H 3465 3955 50  0000 L CNN
+F 1 "1n" H 3465 3955 50  0000 L CNN
 F 2 "" H 3388 3850 50  0001 C CNN
 F 3 "~" H 3350 4000 50  0001 C CNN
@@
 P 3000 3650
 F 0 "R?" V 2793 3650 50  0000 C CNN
-F 1 "1k2" V 2884 3650 50  0000 C CNN
+F 1 "1k5" V 2884 3650 50  0000 C CNN
 F 2 "" V 2930 3650 50  0001 C CNN
 F 3 "~" H 3000 3650 50  0001 C CNN
@@
 P 3000 4200
 F 0 "R?" V 2793 4200 50  0000 C CNN
-F 1 "1k2" V 2884 4200 50  0000 C CNN
+F 1 "820" V 2884 4200 50  0000 C CNN
 F 2 "" V 2930 4200 50  0001 C CNN
 F 3 "~" H 3000 4200 50  0001 C CNN
@@
 P 2450 3650
 F 0 "R?" V 2400 3500 50  0000 C CNN
-F 1 "1k2" V 2550 3600 50  0000 C CNN
+F 1 "820" V 2550 3600 50  0000 C CNN
 F 2 "" V 2380 3650 50  0001 C CNN
 F 3 "~" H 2450 3650 50  0001 C CNN
@@
 P 2450 3400
 F 0 "C?" V 2400 3300 50  0000 C CNN
-F 1 "6n8" V 2500 3550 50  0000 C CNN
+F 1 "3n3" V 2500 3550 50  0000 C CNN
 F 2 "" H 2488 3250 50  0001 C CNN
 F 3 "~" H 2450 3400 50  0001 C CNN
@@
 P 3450 2650
 F 0 "C?" H 3565 2696 50  0000 L CNN
-F 1 "2n2" H 3565 2605 50  0000 L CNN
+F 1 "1n" H 3565 2605 50  0000 L CNN
 F 2 "" H 3488 2500 50  0001 C CNN
 F 3 "~" H 3450 2650 50  0001 C CNN
@@
 P 3000 2950
 F 0 "R?" V 2900 2850 50  0000 C CNN
-F 1 "1k2" V 3100 3000 50  0000 C CNN
+F 1 "1k5" V 3100 3000 50  0000 C CNN
 F 2 "" V 2930 2950 50  0001 C CNN
 F 3 "~" H 3000 2950 50  0001 C CNN
@@
 P 2750 2650
 F 0 "R?" H 2680 2604 50  0000 R CNN
-F 1 "1k2" H 2680 2695 50  0000 R CNN
+F 1 "820" H 2680 2695 50  0000 R CNN
 F 2 "" V 2680 2650 50  0001 C CNN
 F 3 "~" H 2750 2650 50  0001 C CNN
@@
 P 2050 2950
 F 0 "R?" V 1950 2850 50  0000 R CNN
-F 1 "1k2" V 2150 2950 50  0000 R CNN
+F 1 "820" V 2150 2950 50  0000 R CNN
 F 2 "" V 1980 2950 50  0001 C CNN
 F 3 "~" H 2050 2950 50  0001 C CNN
@@
 P 2450 3100
 F 0 "C?" V 2400 3000 50  0000 C CNN
-F 1 "6n8" V 2500 3250 50  0000 C CNN
+F 1 "3n3" V 2500 3250 50  0000 C CNN
 F 2 "" H 2488 2950 50  0001 C CNN
 F 3 "~" H 2450 3100 50  0001 C CNN
@@
 P 3450 6700
 F 0 "C?" H 3565 6746 50  0000 L CNN
-F 1 "2n2" H 3565 6655 50  0000 L CNN
+F 1 "1n" H 3565 6655 50  0000 L CNN
 F 2 "" H 3488 6550 50  0001 C CNN
 F 3 "~" H 3450 6700 50  0001 C CNN
@@
 P 3100 6350
 F 0 "R?" V 2893 6350 50  0000 C CNN
-F 1 "1k2" V 2984 6350 50  0000 C CNN
+F 1 "1k5" V 2984 6350 50  0000 C CNN
 F 2 "" V 3030 6350 50  0001 C CNN
 F 3 "~" H 3100 6350 50  0001 C CNN
@@
 P 3100 6900
 F 0 "R?" V 2893 6900 50  0000 C CNN
-F 1 "1k2" V 2984 6900 50  0000 C CNN
+F 1 "820" V 2984 6900 50  0000 C CNN
 F 2 "" V 3030 6900 50  0001 C CNN
 F 3 "~" H 3100 6900 50  0001 C CNN
@@
 P 2550 6350
 F 0 "R?" V 2500 6200 50  0000 C CNN
-F 1 "1k2" V 2650 6300 50  0000 C CNN
+F 1 "820" V 2650 6300 50  0000 C CNN
 F 2 "" V 2480 6350 50  0001 C CNN
 F 3 "~" H 2550 6350 50  0001 C CNN
@@
 P 2550 6100
 F 0 "C?" V 2500 6000 50  0000 C CNN
-F 1 "6n8" V 2600 6250 50  0000 C CNN
+F 1 "3n3" V 2600 6250 50  0000 C CNN
 F 2 "" H 2588 5950 50  0001 C CNN
 F 3 "~" H 2550 6100 50  0001 C CNN
@@
 P 3550 5350
 F 0 "C?" H 3665 5396 50  0000 L CNN
-F 1 "2n2" H 3665 5305 50  0000 L CNN
+F 1 "1n" H 3665 5305 50  0000 L CNN
 F 2 "" H 3588 5200 50  0001 C CNN
 F 3 "~" H 3550 5350 50  0001 C CNN
@@
 P 3100 5650
 F 0 "R?" V 3000 5550 50  0000 C CNN
-F 1 "1k2" V 3200 5700 50  0000 C CNN
+F 1 "1k5" V 3200 5700 50  0000 C CNN
 F 2 "" V 3030 5650 50  0001 C CNN
 F 3 "~" H 3100 5650 50  0001 C CNN
@@
 P 2850 5350
 F 0 "R?" H 2780 5304 50  0000 R CNN
-F 1 "1k2" H 2780 5395 50  0000 R CNN
+F 1 "820" H 2780 5395 50  0000 R CNN
 F 2 "" V 2780 5350 50  0001 C CNN
 F 3 "~" H 2850 5350 50  0001 C CNN
@@
 P 2150 5650
 F 0 "R?" V 2050 5550 50  0000 R CNN
-F 1 "1k2" V 2250 5650 50  0000 R CNN
+F 1 "820" V 2250 5650 50  0000 R CNN
 F 2 "" V 2080 5650 50  0001 C CNN
 F 3 "~" H 2150 5650 50  0001 C CNN
@@
 P 2550 5800
 F 0 "C?" V 2500 5700 50  0000 C CNN
-F 1 "6n8" V 2600 5950 50  0000 C CNN
+F 1 "3n3" V 2600 5950 50  0000 C CNN
 F 2 "" H 2588 5650 50  0001 C CNN
 F 3 "~" H 2550 5800 50  0001 C CNN
