File: schematics/DykoDAC_Output.sch (KiCad schematic (older format))
At the start: 41 parts

Commit message: finishing
Parts:
- added C49, C51: 100u, Capacitors_SMD:CP_Elec_5x4.5, symbol Device:CP
- added C50, C52: 10u, Capacitors_SMD:C_1206, symbol Device:CP
- C35, C36, C37, C38, C39, C40, C41, C42, C43, C44, C45, C46: renamed from C?; footprint (none) -> Capacitors_SMD:C_1206
- C47, C48, C53, C54: renamed from C?; value C -> 0.1u; footprint (none) -> Capacitors_SMD:C_1206
- J2: renamed from J?; footprint (none) -> Connect:JACK_ALIM
- R10, R11, R12, R13, R14, R15, R16, R17, R18, R19, R20, R21, R22, R23, R24, R25, R26, R7, R8, R9: renamed from R?; footprint (none) -> Resistors_SMD:R_1206
- U10: renamed from U?; footprint (none) -> Housings_SOIC:HSOP-20-1EP_11.0x15.9mm_Pitch1.27mm_SlugDown
- U9: renamed from U?; footprint (none) -> Housings_SOIC:SOIC-8_3.9x4.9mm_Pitch1.27mm
Connections:
- wire segments 140 -> 154

Commit message: changed filter values started with PCB design
Parts:
- C35, C42: value 4.7u -> 10u
- C37, C38, C40, C41: value 6n8 -> 3n3
- C43, C44, C45, C46: value 2n2 -> 1n
- R10, R11, R12, R15, R18, R7, R8, R9: value 1k2 -> 820
- R13, R14, R16, R17: value 1k2 -> 1k5
Changed lines of the file:
@@
 P 2700 1250
 F 0 "C42" H 2800 1350 50  0000 C CNN
-F 1 "4.7u" H 2800 1150 50  0000 C CNN
+F 1 "10u" H 2800 1150 50  0000 C CNN
 F 2 "Capacitors_SMD:C_1206" H 2738 1100 50  0001 C CNN
 F 3 "~" H 2700 1250 50  0001 C CNN
@@
 P 1350 1250
 F 0 "C35" H 1450 1150 50  0000 C CNN
-F 1 "4.7u" H 1450 1350 50  0000 C CNN
+F 1 "10u" H 1450 1350 50  0000 C CNN
 F 2 "Capacitors_SMD:C_1206" H 1388 1100 50  0001 C CNN
 F 3 "~" H 1350 1250 50  0001 C CNN
@@
 P 3350 4000
 F 0 "C43" H 3465 4046 50  0000 L CNN
-F 1 "2n2" H 3465 3955 50  0000 L CNN
+F 1 "1n" H 3465 3955 50  0000 L CNN
 F 2 "Capacitors_SMD:C_1206" H 3388 3850 50  0001 C CNN
 F 3 "~" H 3350 4000 50  0001 C CNN
@@
 P 3000 3650
 F 0 "R14" V 2793 3650 50  0000 C CNN
-F 1 "1k2" V 2884 3650 50  0000 C CNN
+F 1 "1k5" V 2884 3650 50  0000 C CNN
 F 2 "Resistors_SMD:R_1206" V 2930 3650 50  0001 C CNN
 F 3 "~" H 3000 3650 50  0001 C CNN
@@
 P 3000 4200
 F 0 "R15" V 2793 4200 50  0000 C CNN
-F 1 "1k2" V 2884 4200 50  0000 C CNN
+F 1 "820" V 2884 4200 50  0000 C CNN
 F 2 "Resistors_SMD:R_1206" V 2930 4200 50  0001 C CNN
 F 3 "~" H 3000 4200 50  0001 C CNN
@@
 P 2450 3650
 F 0 "R9" V 2400 3500 50  0000 C CNN
-F 1 "1k2" V 2550 3600 50  0000 C CNN
+F 1 "820" V 2550 3600 50  0000 C CNN
 F 2 "Resistors_SMD:R_1206" V 2380 3650 50  0001 C CNN
 F 3 "~" H 2450 3650 50  0001 C CNN
@@
 P 2450 3400
 F 0 "C38" V 2400 3250 50  0000 C CNN
-F 1 "6n8" V 2500 3550 50  0000 C CNN
+F 1 "3n3" V 2500 3550 50  0000 C CNN
 F 2 "Capacitors_SMD:C_1206" H 2488 3250 50  0001 C CNN
 F 3 "~" H 2450 3400 50  0001 C CNN
@@
 P 3450 2650
 F 0 "C44" H 3565 2696 50  0000 L CNN
-F 1 "2n2" H 3565 2605 50  0000 L CNN
+F 1 "1n" H 3565 2605 50  0000 L CNN
 F 2 "Capacitors_SMD:C_1206" H 3488 2500 50  0001 C CNN
 F 3 "~" H 3450 2650 50  0001 C CNN
@@
 P 3000 2950
 F 0 "R13" V 2900 2850 50  0000 C CNN
-F 1 "1k2" V 3100 3000 50  0000 C CNN
+F 1 "1k5" V 3100 3000 50  0000 C CNN
 F 2 "Resistors_SMD:R_1206" V 2930 2950 50  0001 C CNN
 F 3 "~" H 3000 2950 50  0001 C CNN
@@
 P 2750 2650
 F 0 "R11" H 2680 2604 50  0000 R CNN
-F 1 "1k2" H 2680 2695 50  0000 R CNN
+F 1 "820" H 2680 2695 50  0000 R CNN
 F 2 "Resistors_SMD:R_1206" V 2680 2650 50  0001 C CNN
 F 3 "~" H 2750 2650 50  0001 C CNN
@@
 P 2050 2950
 F 0 "R7" V 1950 2850 50  0000 R CNN
-F 1 "1k2" V 2150 2950 50  0000 R CNN
+F 1 "820" V 2150 2950 50  0000 R CNN
 F 2 "Resistors_SMD:R_1206" V 1980 2950 50  0001 C CNN
 F 3 "~" H 2050 2950 50  0001 C CNN
@@
 P 2450 3100
 F 0 "C37" V 2400 2950 50  0000 C CNN
-F 1 "6n8" V 2500 3250 50  0000 C CNN
+F 1 "3n3" V 2500 3250 50  0000 C CNN
 F 2 "Capacitors_SMD:C_1206" H 2488 2950 50  0001 C CNN
 F 3 "~" H 2450 3100 50  0001 C CNN
@@
 P 3450 6700
 F 0 "C45" H 3565 6746 50  0000 L CNN
-F 1 "2n2" H 3565 6655 50  0000 L CNN
+F 1 "1n" H 3565 6655 50  0000 L CNN
 F 2 "Capacitors_SMD:C_1206" H 3488 6550 50  0001 C CNN
 F 3 "~" H 3450 6700 50  0001 C CNN
@@
 P 3100 6350
 F 0 "R17" V 2893 6350 50  0000 C CNN
-F 1 "1k2" V 2984 6350 50  0000 C CNN
+F 1 "1k5" V 2984 6350 50  0000 C CNN
 F 2 "Resistors_SMD:R_1206" V 3030 6350 50  0001 C CNN
 F 3 "~" H 3100 6350 50  0001 C CNN
@@
 P 3100 6900
 F 0 "R18" V 2893 6900 50  0000 C CNN
-F 1 "1k2" V 2984 6900 50  0000 C CNN
+F 1 "820" V 2984 6900 50  0000 C CNN
 F 2 "Resistors_SMD:R_1206" V 3030 6900 50  0001 C CNN
 F 3 "~" H 3100 6900 50  0001 C CNN
@@
 P 2550 6350
 F 0 "R10" V 2500 6150 50  0000 C CNN
-F 1 "1k2" V 2650 6300 50  0000 C CNN
+F 1 "820" V 2650 6300 50  0000 C CNN
 F 2 "Resistors_SMD:R_1206" V 2480 6350 50  0001 C CNN
 F 3 "~" H 2550 6350 50  0001 C CNN
@@
 P 2550 6100
 F 0 "C41" V 2500 5950 50  0000 C CNN
-F 1 "6n8" V 2600 6250 50  0000 C CNN
+F 1 "3n3" V 2600 6250 50  0000 C CNN
 F 2 "Capacitors_SMD:C_1206" H 2588 5950 50  0001 C CNN
 F 3 "~" H 2550 6100 50  0001 C CNN
@@
 P 3550 5350
 F 0 "C46" H 3665 5396 50  0000 L CNN
-F 1 "2n2" H 3665 5305 50  0000 L CNN
+F 1 "1n" H 3665 5305 50  0000 L CNN
 F 2 "Capacitors_SMD:C_1206" H 3588 5200 50  0001 C CNN
 F 3 "~" H 3550 5350 50  0001 C CNN
@@
 P 3100 5650
 F 0 "R16" V 3000 5550 50  0000 C CNN
-F 1 "1k2" V 3200 5700 50  0000 C CNN
+F 1 "1k5" V 3200 5700 50  0000 C CNN
 F 2 "Resistors_SMD:R_1206" V 3030 5650 50  0001 C CNN
 F 3 "~" H 3100 5650 50  0001 C CNN
@@
 P 2850 5350
 F 0 "R12" H 2780 5304 50  0000 R CNN
-F 1 "1k2" H 2780 5395 50  0000 R CNN
+F 1 "820" H 2780 5395 50  0000 R CNN
 F 2 "Resistors_SMD:R_1206" V 2780 5350 50  0001 C CNN
 F 3 "~" H 2850 5350 50  0001 C CNN
@@
 P 2150 5650
 F 0 "R8" V 2050 5550 50  0000 R CNN
-F 1 "1k2" V 2250 5650 50  0000 R CNN
+F 1 "820" V 2250 5650 50  0000 R CNN
 F 2 "Resistors_SMD:R_1206" V 2080 5650 50  0001 C CNN
 F 3 "~" H 2150 5650 50  0001 C CNN
@@
 P 2550 5800
 F 0 "C40" V 2500 5650 50  0000 C CNN
-F 1 "6n8" V 2600 5950 50  0000 C CNN
+F 1 "3n3" V 2600 5950 50  0000 C CNN
 F 2 "Capacitors_SMD:C_1206" H 2588 5650 50  0001 C CNN
 F 3 "~" H 2550 5800 50  0001 C CNN
@@
 L power:+9V #PWR037
 U 1 1 5CD91CF9
-P 7600 2200
-F 0 "#PWR037" H 7600 2050 50  0001 C CNN
-F 1 "+9V" H 7615 2373 50  0000 C CNN
-F 2 "" H 7600 2200 50  0001 C CNN
-F 3 "" H 7600 2200 50  0001 C CNN
-	1    7600 2200
+P 7600 2450
+F 0 "#PWR037" H 7600 2300 50  0001 C CNN
+F 1 "+9V" H 7615 2623 50  0000 C CNN
+F 2 "" H 7600 2450 50  0001 C CNN
+F 3 "" H 7600 2450 50  0001 C CNN
+	1    7600 2450
 	1    0    0    -1
 $EndComp
@@
 L power:-9V #PWR040
 U 1 1 5CDCF6C9
-P 9150 2200
-F 0 "#PWR040" H 9150 2075 50  0001 C CNN
-F 1 "-9V" H 9165 2373 50  0000 C CNN
-F 2 "" H 9150 2200 50  0001 C CNN
-F 3 "" H 9150 2200 50  0001 C CNN
-	1    9150 2200
+P 9150 2450
+F 0 "#PWR040" H 9150 2325 50  0001 C CNN
+F 1 "-9V" H 9165 2623 50  0000 C CNN
+F 2 "" H 9150 2450 50  0001 C CNN
+F 3 "" H 9150 2450 50  0001 C CNN
+	1    9150 2450
 	1    0    0    -1
 $EndComp
@@
 Wire Wire Line
 	9750 3250 9950 3250
-$Comp
-L Device:CP C49
-U 1 1 5D14BCCD
-P 7950 2350
-F 0 "C49" V 8000 2500 50  0000 C CNN
-F 1 "100u" V 8000 2200 50  0000 C CNN
-F 2 "Capacitors_SMD:CP_Elec_5x4.5" H 7988 2200 50  0001 C CNN
-F 3 "~" H 7950 2350 50  0001 C CNN
-	1    7950 2350
-	0    -1   -1   0
-$EndComp
 $Comp
 L Device:CP C50
@@
 $EndComp
 $Comp
-L Device:CP C51
-U 1 1 5D14DFA3
-P 8850 2350
-F 0 "C51" V 8900 2500 50  0000 C CNN
-F 1 "100u" V 8900 2200 50  0000 C CNN
-F 2 "Capacitors_SMD:CP_Elec_5x4.5" H 8888 2200 50  0001 C CNN
-F 3 "~" H 8850 2350 50  0001 C CNN
-	1    8850 2350
-	0    -1   -1   0
-$EndComp
-$Comp
 L Device:CP C52
 U 1 1 5D14EBD1
@@
 $EndComp
 Wire Wire Line
-	8100 2700 8350 2700
-Wire Wire Line
-	7600 2200 7600 2350
-Wire Wire Line
-	9150 2200 9150 2350
-Wire Wire Line
-	9150 2350 9000 2350
-Wire Wire Line
-	8100 2350 8350 2350
-Wire Wire Line
-	9150 2350 9150 2700
-Connection ~ 9150 2350
-Wire Wire Line
 	9000 2700 9150 2700
-Connection ~ 9150 2700
 Wire Wire Line
 	9150 2700 9150 3000
 Wire Wire Line
 	7800 2700 7600 2700
-Connection ~ 7600 2700
 Wire Wire Line
 	7600 2700 7600 3100
-Wire Wire Line
-	7800 2350 7600 2350
-Connection ~ 7600 2350
-Wire Wire Line
-	7600 2350 7600 2700
 $Comp
 L power:GND #PWR038
 U 1 1 5D17DB7D
-P 8350 2200
-F 0 "#PWR038" H 8350 1950 50  0001 C CNN
-F 1 "GND" H 8355 2027 50  0000 C CNN
-F 2 "" H 8350 2200 50  0001 C CNN
-F 3 "" H 8350 2200 50  0001 C CNN
-	1    8350 2200
+P 8350 2450
+F 0 "#PWR038" H 8350 2200 50  0001 C CNN
+F 1 "GND" H 8355 2277 50  0000 C CNN
+F 2 "" H 8350 2450 50  0001 C CNN
+F 3 "" H 8350 2450 50  0001 C CNN
+	1    8350 2450
 	-1   0    0    1
 $EndComp
-Wire Wire Line
-	8350 2200 8350 2350
-Connection ~ 8350 2350
-Wire Wire Line
-	8350 2350 8700 2350
-Wire Wire Line
-	8350 2700 8350 2350
+$Comp
+L power:+9V #PWR0101
+U 1 1 5D188C88
+P 4750 1100
+F 0 "#PWR0101" H 4750 950 50  0001 C CNN
+F 1 "+9V" H 4765 1273 50  0000 C CNN
+F 2 "" H 4750 1100 50  0001 C CNN
+F 3 "" H 4750 1100 50  0001 C CNN
+	1    4750 1100
+	1    0    0    -1
+$EndComp
+$Comp
+L power:-9V #PWR0102
+U 1 1 5D188C8E
+P 6300 1100
+F 0 "#PWR0102" H 6300 975 50  0001 C CNN
+F 1 "-9V" H 6315 1273 50  0000 C CNN
+F 2 "" H 6300 1100 50  0001 C CNN
+F 3 "" H 6300 1100 50  0001 C CNN
+	1    6300 1100
+	1    0    0    -1
+$EndComp
+$Comp
+L Device:CP C49
+U 1 1 5D188C94
+P 5100 1250
+F 0 "C49" V 5150 1400 50  0000 C CNN
+F 1 "100u" V 5150 1100 50  0000 C CNN
+F 2 "Capacitors_SMD:CP_Elec_5x4.5" H 5138 1100 50  0001 C CNN
+F 3 "~" H 5100 1250 50  0001 C CNN
+	1    5100 1250
+	0    -1   -1   0
+$EndComp
+$Comp
+L Device:CP C51
+U 1 1 5D188C9A
+P 6000 1250
+F 0 "C51" V 6050 1400 50  0000 C CNN
+F 1 "100u" V 6050 1100 50  0000 C CNN
+F 2 "Capacitors_SMD:CP_Elec_5x4.5" H 6038 1100 50  0001 C CNN
+F 3 "~" H 6000 1250 50  0001 C CNN
+	1    6000 1250
+	0    -1   -1   0
+$EndComp
+Wire Wire Line
+	4750 1100 4750 1250
+Wire Wire Line
+	6300 1100 6300 1250
+Wire Wire Line
+	6300 1250 6150 1250
+Wire Wire Line
+	5250 1250 5500 1250
+Wire Wire Line
+	4950 1250 4750 1250
+$Comp
+L power:GND #PWR0103
+U 1 1 5D188CA9
+P 5500 1100
+F 0 "#PWR0103" H 5500 850 50  0001 C CNN
+F 1 "GND" H 5505 927 50  0000 C CNN
+F 2 "" H 5500 1100 50  0001 C CNN
+F 3 "" H 5500 1100 50  0001 C CNN
+	1    5500 1100
+	-1   0    0    1
+$EndComp
+Wire Wire Line
+	5500 1100 5500 1250
+Connection ~ 5500 1250
+Wire Wire Line
+	5500 1250 5850 1250
+Wire Wire Line
+	8100 2700 8350 2700
+Wire Wire Line
+	7600 2700 7600 2450
+Connection ~ 7600 2700
+Wire Wire Line
+	8350 2450 8350 2700
 Connection ~ 8350 2700
 Wire Wire Line
 	8350 2700 8700 2700
+Wire Wire Line
+	9150 2450 9150 2700
+Connection ~ 9150 2700
 $EndSCHEMATC

Commit message: lots of stuf ....
Parts:
- C35, C36, C37, C38, C39, C40, C41, C42, C43, C44, C45, C46, C47, C48, C50, C52, C53, C54: footprint Capacitors_SMD:C_1206 -> Capacitors_SMD:C_0603_HandSoldering
- R10, R11, R12, R13, R14, R15, R16, R17, R18, R19, R20, R21, R22, R23, R24, R25, R26, R7, R8, R9: footprint Resistors_SMD:R_1206 -> Resistors_SMD:R_0603_HandSoldering
Other:
- moved on the sheet: C43, C45, R10, R15, R18, R19, R20, R9

Commit message: no message
Parts:
- C35, C42, C50, C52: footprint Capacitors_SMD:C_0603_HandSoldering -> Capacitors_SMD:CP_Elec_4x5.7
- C36, C37, C38, C39, C40, C41, C43, C44, C45, C46, C47, C48, C53, C54: footprint Capacitors_SMD:C_0603_HandSoldering -> Capacitors_SMD:C_0603
- R10, R11, R12, R13, R14, R15, R16, R17, R18, R19, R20, R21, R22, R23, R24, R25, R26, R7, R8, R9: footprint Resistors_SMD:R_0603_HandSoldering -> Resistors_SMD:R_0603
- U10: value TPA6120 -> TPA6120A2

Commit message: opamp filter pcb
Parts:
- removed J2: AudioJack3, Connect:JACK_ALIM, symbol Connector:AudioJack3
- added J2: AudioJack2_Ground_Switch, Connect:Stereo_Jack_3.5mm_Switch_Ledino_KB3SPRS, symbol kamtar:AudioJack2_Ground_Switch
- C35, C42, C50, C52: footprint Capacitors_SMD:CP_Elec_4x5.7 -> Capacitors_Tantalum_SMD:CP_Tantalum_Case-A_EIA-3216-18_Reflow
- C49, C51: footprint Capacitors_SMD:CP_Elec_5x4.5 -> Capacitors_Tantalum_SMD:CP_Tantalum_Case-D_EIA-7343-31_Reflow
- U10: footprint Housings_SOIC:HSOP-20-1EP_11.0x15.9mm_Pitch1.27mm_SlugDown -> test:SOIC-20W_ThermalPad
Connections:
- wire segments 154 -> 153
- no-connect marks 0 -> 2
Changed lines of the file:
@@
 F 0 "C42" H 2800 1350 50  0000 C CNN
 F 1 "10u" H 2800 1150 50  0000 C CNN
-F 2 "Capacitors_SMD:CP_Elec_4x5.7" H 2738 1100 50  0001 C CNN
+F 2 "Capacitors_Tantalum_SMD:CP_Tantalum_Case-A_EIA-3216-18_Reflow" H 2738 1100 50  0001 C CNN
 F 3 "~" H 2700 1250 50  0001 C CNN
 	1    2700 1250
@@
 F 0 "C35" H 1450 1150 50  0000 C CNN
 F 1 "10u" H 1450 1350 50  0000 C CNN
-F 2 "Capacitors_SMD:CP_Elec_4x5.7" H 1388 1100 50  0001 C CNN
+F 2 "Capacitors_Tantalum_SMD:CP_Tantalum_Case-A_EIA-3216-18_Reflow" H 1388 1100 50  0001 C CNN
 F 3 "~" H 1350 1250 50  0001 C CNN
 	1    1350 1250
@@
 F 0 "U10" H 8375 3337 60  0000 C CNN
 F 1 "TPA6120A2" H 8375 3231 60  0000 C CNN
-F 2 "Housings_SOIC:HSOP-20-1EP_11.0x15.9mm_Pitch1.27mm_SlugDown" H 8000 3150 60  0001 C CNN
+F 2 "test:SOIC-20W_ThermalPad" H 8000 3150 60  0001 C CNN
 F 3 "" H 8000 3150 60  0001 C CNN
 	1    8000 3150
@@
 	7150 4700 7150 4750
 $Comp
-L Connector:AudioJack3 J2
-U 1 1 5CD64FCC
-P 10400 3700
-F 0 "J2" H 10120 3633 50  0000 R CNN
-F 1 "AudioJack3" H 10120 3724 50  0000 R CNN
-F 2 "Connect:JACK_ALIM" H 10400 3700 50  0001 C CNN
-F 3 "~" H 10400 3700 50  0001 C CNN
-	1    10400 3700
-	-1   0    0    1
-$EndComp
-$Comp
 L power:GND #PWR042
 U 1 1 5CD6B3CD
-P 10000 3900
-F 0 "#PWR042" H 10000 3650 50  0001 C CNN
-F 1 "GND" H 10005 3727 50  0000 C CNN
-F 2 "" H 10000 3900 50  0001 C CNN
-F 3 "" H 10000 3900 50  0001 C CNN
-	1    10000 3900
-	1    0    0    -1
-$EndComp
-Wire Wire Line
-	10000 3900 10000 3800
-Wire Wire Line
-	10000 3800 10200 3800
+P 10600 4200
+F 0 "#PWR042" H 10600 3950 50  0001 C CNN
+F 1 "GND" H 10605 4027 50  0000 C CNN
+F 2 "" H 10600 4200 50  0001 C CNN
+F 3 "" H 10600 4200 50  0001 C CNN
+	1    10600 4200
+	1    0    0    -1
+$EndComp
+Wire Wire Line
+	10600 4200 10600 4100
 $Comp
 L power:GND #PWR039
@@
 	9100 4000 9350 4000
 Connection ~ 9100 4000
-Wire Wire Line
-	9650 3600 10200 3600
-Wire Wire Line
-	9650 4000 9800 4000
-Wire Wire Line
-	9800 4000 9800 3700
-Wire Wire Line
-	9800 3700 10200 3700
 $Comp
 L Device:C C48
@@
 F 0 "C50" V 8000 2850 50  0000 C CNN
 F 1 "10u" V 8000 2550 50  0000 C CNN
-F 2 "Capacitors_SMD:CP_Elec_4x5.7" H 7988 2550 50  0001 C CNN
+F 2 "Capacitors_Tantalum_SMD:CP_Tantalum_Case-A_EIA-3216-18_Reflow" H 7988 2550 50  0001 C CNN
 F 3 "~" H 7950 2700 50  0001 C CNN
 	1    7950 2700
@@
 F 0 "C52" V 8900 2850 50  0000 C CNN
 F 1 "10u" V 8900 2550 50  0000 C CNN
-F 2 "Capacitors_SMD:CP_Elec_4x5.7" H 8888 2550 50  0001 C CNN
+F 2 "Capacitors_Tantalum_SMD:CP_Tantalum_Case-A_EIA-3216-18_Reflow" H 8888 2550 50  0001 C CNN
 F 3 "~" H 8850 2700 50  0001 C CNN
 	1    8850 2700
@@
 F 0 "C49" V 5150 1400 50  0000 C CNN
 F 1 "100u" V 5150 1100 50  0000 C CNN
-F 2 "Capacitors_SMD:CP_Elec_5x4.5" H 5138 1100 50  0001 C CNN
+F 2 "Capacitors_Tantalum_SMD:CP_Tantalum_Case-D_EIA-7343-31_Reflow" H 5138 1100 50  0001 C CNN
 F 3 "~" H 5100 1250 50  0001 C CNN
 	1    5100 1250
@@
 F 0 "C51" V 6050 1400 50  0000 C CNN
 F 1 "100u" V 6050 1100 50  0000 C CNN
-F 2 "Capacitors_SMD:CP_Elec_5x4.5" H 6038 1100 50  0001 C CNN
+F 2 "Capacitors_Tantalum_SMD:CP_Tantalum_Case-D_EIA-7343-31_Reflow" H 6038 1100 50  0001 C CNN
 F 3 "~" H 6000 1250 50  0001 C CNN
 	1    6000 1250
@@
 	4400 3550 4200 3550
 Connection ~ 4200 3550
+$Comp
+L kamtar:AudioJack2_Ground_Switch J2
+U 1 1 5E5732C1
+P 10600 3800
+F 0 "J2" H 10420 3818 50  0000 R CNN
+F 1 "AudioJack2_Ground_Switch" H 10420 3727 50  0000 R CNN
+F 2 "Connect:Stereo_Jack_3.5mm_Switch_Ledino_KB3SPRS" H 10600 4000 50  0001 C CNN
+F 3 "~" H 10600 4000 50  0001 C CNN
+	1    10600 3800
+	-1   0    0    -1
+$EndComp
+Wire Wire Line
+	9650 3600 10400 3600
+NoConn ~ 10400 3700
+NoConn ~ 10400 3900
+Wire Wire Line
+	10200 4000 10200 3800
+Wire Wire Line
+	10200 3800 10400 3800
+Wire Wire Line
+	9650 4000 10200 4000
 $EndSCHEMATC

Commit message: pcb update
Parts:
- J2: value AudioJack2_Ground_Switch -> AudioJack
Changed lines of the file:
@@
 P 10600 3800
 F 0 "J2" H 10420 3818 50  0000 R CNN
-F 1 "AudioJack2_Ground_Switch" H 10420 3727 50  0000 R CNN
+F 1 "AudioJack" H 10420 3727 50  0000 R CNN
 F 2 "Connect:Stereo_Jack_3.5mm_Switch_Ledino_KB3SPRS" H 10600 4000 50  0001 C CNN
 F 3 "~" H 10600 4000 50  0001 C CNN

Commit message: pcb
Parts:
- removed C49, C51: 100u, Capacitors_Tantalum_SMD:CP_Tantalum_Case-D_EIA-7343-31_Reflow, symbol Device:CP
Connections:
- wire segments 153 -> 146
Changed lines of the file:
@@
-	-1   0    0    1
-$EndComp
-$Comp
-L power:+9V #PWR0101
-U 1 1 5D188C88
-P 4750 1100
-F 0 "#PWR0101" H 4750 950 50  0001 C CNN
-F 1 "+9V" H 4765 1273 50  0000 C CNN
-F 2 "" H 4750 1100 50  0001 C CNN
-F 3 "" H 4750 1100 50  0001 C CNN
-	1    4750 1100
-	1    0    0    -1
-$EndComp
-$Comp
-L power:-9V #PWR0102
-U 1 1 5D188C8E
-P 6300 1100
-F 0 "#PWR0102" H 6300 975 50  0001 C CNN
-F 1 "-9V" H 6315 1273 50  0000 C CNN
-F 2 "" H 6300 1100 50  0001 C CNN
-F 3 "" H 6300 1100 50  0001 C CNN
-	1    6300 1100
-	1    0    0    -1
-$EndComp
-$Comp
-L Device:CP C49
-U 1 1 5D188C94
-P 5100 1250
-F 0 "C49" V 5150 1400 50  0000 C CNN
-F 1 "100u" V 5150 1100 50  0000 C CNN
-F 2 "Capacitors_Tantalum_SMD:CP_Tantalum_Case-D_EIA-7343-31_Reflow" H 5138 1100 50  0001 C CNN
-F 3 "~" H 5100 1250 50  0001 C CNN
-	1    5100 1250
-	0    -1   -1   0
-$EndComp
-$Comp
-L Device:CP C51
-U 1 1 5D188C9A
-P 6000 1250
-F 0 "C51" V 6050 1400 50  0000 C CNN
-F 1 "100u" V 6050 1100 50  0000 C CNN
-F 2 "Capacitors_Tantalum_SMD:CP_Tantalum_Case-D_EIA-7343-31_Reflow" H 6038 1100 50  0001 C CNN
-F 3 "~" H 6000 1250 50  0001 C CNN
-	1    6000 1250
-	0    -1   -1   0
-$EndComp
-Wire Wire Line
-	4750 1100 4750 1250
-Wire Wire Line
-	6300 1100 6300 1250
-Wire Wire Line
-	6300 1250 6150 1250
-Wire Wire Line
-	5250 1250 5500 1250
-Wire Wire Line
-	4950 1250 4750 1250
-$Comp
-L power:GND #PWR0103
-U 1 1 5D188CA9
-P 5500 1100
-F 0 "#PWR0103" H 5500 850 50  0001 C CNN
-F 1 "GND" H 5505 927 50  0000 C CNN
-F 2 "" H 5500 1100 50  0001 C CNN
-F 3 "" H 5500 1100 50  0001 C CNN
-	1    5500 1100
 	-1   0    0    1
 $EndComp
 Wire Wire Line
-	5500 1100 5500 1250
-Connection ~ 5500 1250
-Wire Wire Line
-	5500 1250 5850 1250
-Wire Wire Line
 	8100 2700 8350 2700

Commit message: pcb
Parts:
- added TP1: TestPoint, Connect:1pin, symbol Connector:TestPoint
Connections:
- wire segments 146 -> 147
Changed lines of the file:
@@
 Wire Wire Line
 	9650 4000 10200 4000
+$Comp
+L Connector:TestPoint TP1
+U 1 1 5E58C58D
+P 8500 1500
+F 0 "TP1" H 8558 1618 50  0000 L CNN
+F 1 "TestPoint" H 8558 1527 50  0000 L CNN
+F 2 "Connect:1pin" H 8700 1500 50  0001 C CNN
+F 3 "~" H 8700 1500 50  0001 C CNN
+	1    8500 1500
+	1    0    0    -1
+$EndComp
+$Comp
+L power:GND #PWR062
+U 1 1 5E58D3F2
+P 8500 1650
+F 0 "#PWR062" H 8500 1400 50  0001 C CNN
+F 1 "GND" H 8505 1477 50  0000 C CNN
+F 2 "" H 8500 1650 50  0001 C CNN
+F 3 "" H 8500 1650 50  0001 C CNN
+	1    8500 1650
+	1    0    0    -1
+$EndComp
+Wire Wire Line
+	8500 1650 8500 1500
 $EndSCHEMATC
