File: schematics/DykoDAC_Output.sch (KiCad schematic (older format))
At the start: 42 parts, among them J2 AudioJack, U10 TPA6120A2, U9 AD8620

Commit message: minor chages
Parts:
- J2: symbol kamtar:AudioJack2_Ground_Switch -> DykoDAC-rescue:AudioJack2_Ground_Switch-kamtar
- U10: symbol ti:TPA6120 -> DykoDAC-rescue:TPA6120-ti
Changed lines of the file:
@@
 Filter and headphone amp
 $Comp
-L ti:TPA6120 U10
+L DykoDAC-rescue:TPA6120-ti U10
 U 1 1 5CD23F1B
 P 8000 3150
+AR Path="/5CD23F1B" Ref="U10"  Part="1"
+AR Path="/5C90E752/5CD23F1B" Ref="U10"  Part="1"
 F 0 "U10" H 8375 3337 60  0000 C CNN
 F 1 "TPA6120A2" H 8375 3231 60  0000 C CNN
@@
 Connection ~ 4200 3550
 $Comp
-L kamtar:AudioJack2_Ground_Switch J2
+L DykoDAC-rescue:AudioJack2_Ground_Switch-kamtar J2
 U 1 1 5E5732C1
 P 10600 3800
+AR Path="/5E5732C1" Ref="J2"  Part="1"
+AR Path="/5C90E752/5E5732C1" Ref="J2"  Part="1"
 F 0 "J2" H 10420 3818 50  0000 R CNN
 F 1 "AudioJack" H 10420 3727 50  0000 R CNN

Commit message: first revision finished
Parts:
- TP1: footprint Connect:1pin -> TestPoint:TestPoint_Plated_Hole_D2.0mm
Changed lines of the file:
@@
 F 0 "TP1" H 8558 1618 50  0000 L CNN
 F 1 "TestPoint" H 8558 1527 50  0000 L CNN
-F 2 "Connect:1pin" H 8700 1500 50  0001 C CNN
+F 2 "TestPoint:TestPoint_Plated_Hole_D2.0mm" H 8700 1500 50  0001 C CNN
 F 3 "~" H 8700 1500 50  0001 C CNN
 	1    8500 1500

Commit message: update
Parts:
- C35, C42, C50, C52: footprint Capacitors_Tantalum_SMD:CP_Tantalum_Case-A_EIA-3216-18_Reflow -> Capacitor_Tantalum_SMD:CP_EIA-3216-18_Kemet-A
- J2: footprint Connect:Stereo_Jack_3.5mm_Switch_Ledino_KB3SPRS -> kamtar:StereoJack_3.5mm_Lumberg
Changed lines of the file:
@@
 F 0 "C42" H 2800 1350 50  0000 C CNN
 F 1 "10u" H 2800 1150 50  0000 C CNN
-F 2 "Capacitors_Tantalum_SMD:CP_Tantalum_Case-A_EIA-3216-18_Reflow" H 2738 1100 50  0001 C CNN
+F 2 "Capacitor_Tantalum_SMD:CP_EIA-3216-18_Kemet-A" H 2738 1100 50  0001 C CNN
 F 3 "~" H 2700 1250 50  0001 C CNN
 	1    2700 1250
@@
 F 0 "C35" H 1450 1150 50  0000 C CNN
 F 1 "10u" H 1450 1350 50  0000 C CNN
-F 2 "Capacitors_Tantalum_SMD:CP_Tantalum_Case-A_EIA-3216-18_Reflow" H 1388 1100 50  0001 C CNN
+F 2 "Capacitor_Tantalum_SMD:CP_EIA-3216-18_Kemet-A" H 1388 1100 50  0001 C CNN
 F 3 "~" H 1350 1250 50  0001 C CNN
 	1    1350 1250
@@
 F 0 "C50" V 8000 2850 50  0000 C CNN
 F 1 "10u" V 8000 2550 50  0000 C CNN
-F 2 "Capacitors_Tantalum_SMD:CP_Tantalum_Case-A_EIA-3216-18_Reflow" H 7988 2550 50  0001 C CNN
+F 2 "Capacitor_Tantalum_SMD:CP_EIA-3216-18_Kemet-A" H 7988 2550 50  0001 C CNN
 F 3 "~" H 7950 2700 50  0001 C CNN
 	1    7950 2700
@@
 F 0 "C52" V 8900 2850 50  0000 C CNN
 F 1 "10u" V 8900 2550 50  0000 C CNN
-F 2 "Capacitors_Tantalum_SMD:CP_Tantalum_Case-A_EIA-3216-18_Reflow" H 8888 2550 50  0001 C CNN
+F 2 "Capacitor_Tantalum_SMD:CP_EIA-3216-18_Kemet-A" H 8888 2550 50  0001 C CNN
 F 3 "~" H 8850 2700 50  0001 C CNN
 	1    8850 2700
@@
 F 0 "J2" H 10420 3818 50  0000 R CNN
 F 1 "AudioJack" H 10420 3727 50  0000 R CNN
-F 2 "Connect:Stereo_Jack_3.5mm_Switch_Ledino_KB3SPRS" H 10600 4000 50  0001 C CNN
+F 2 "kamtar:StereoJack_3.5mm_Lumberg" H 10600 4000 50  0001 C CNN
 F 3 "~" H 10600 4000 50  0001 C CNN
 	1    10600 3800

Commit message: 9V -> 12V symbol
Parts:
- U9: value AD8620 -> AD8620/AD712
Connections:
- net labels added: +12V, -12V
- net labels removed: +9V, -9V
Changed lines of the file:
@@
 P 3850 3550
 F 0 "U9" H 3850 3917 50  0000 C CNN
-F 1 "AD8620" H 3850 3826 50  0000 C CNN
+F 1 "AD8620/AD712" H 3850 3826 50  0000 C CNN
 F 2 "Housings_SOIC:SOIC-8_3.9x4.9mm_Pitch1.27mm" H 3850 3550 50  0001 C CNN
 F 3 "http://www.analog.com/media/en/technical-documentation/data-sheets/AD8610_8620.pdf" H 3850 3550 50  0001 C CNN
@@
 P 2000 1100
 F 0 "U9" V 2100 1100 50  0000 L CNN
-F 1 "AD8620" V 2000 950 50  0000 L CNN
+F 1 "AD8620/AD712" V 2000 850 50  0000 L CNN
 F 2 "Housings_SOIC:SOIC-8_3.9x4.9mm_Pitch1.27mm" H 2000 1100 50  0001 C CNN
 F 3 "http://www.analog.com/media/en/technical-documentation/data-sheets/AD8610_8620.pdf" H 2000 1100 50  0001 C CNN
@@
 U 1 1 5C911381
 P 2500 1250
-F 0 "C39" H 2600 1150 50  0000 C CNN
-F 1 "0.1u" H 2600 1350 50  0000 C CNN
+F 0 "C39" H 2600 1350 50  0000 C CNN
+F 1 "0.1u" H 2600 1450 50  0000 C CNN
 F 2 "Capacitors_SMD:C_0603" H 2538 1100 50  0001 C CNN
 F 3 "~" H 2500 1250 50  0001 C CNN
@@
 U 1 1 5C91151E
 P 2700 1250
-F 0 "C42" H 2800 1350 50  0000 C CNN
-F 1 "10u" H 2800 1150 50  0000 C CNN
+F 0 "C42" H 2800 1150 50  0000 C CNN
+F 1 "10u" H 2800 1050 50  0000 C CNN
 F 2 "Capacitor_Tantalum_SMD:CP_EIA-3216-18_Kemet-A" H 2738 1100 50  0001 C CNN
 F 3 "~" H 2700 1250 50  0001 C CNN
@@
 U 1 1 5C911889
 P 1550 1250
-F 0 "C36" H 1450 1150 50  0000 C CNN
-F 1 "0.1u" H 1450 1350 50  0000 C CNN
+F 0 "C36" H 1450 1350 50  0000 C CNN
+F 1 "0.1u" H 1450 1450 50  0000 C CNN
 F 2 "Capacitors_SMD:C_0603" H 1588 1100 50  0001 C CNN
 F 3 "~" H 1550 1250 50  0001 C CNN
@@
 U 1 1 5C911890
 P 1350 1250
-F 0 "C35" H 1450 1150 50  0000 C CNN
-F 1 "10u" H 1450 1350 50  0000 C CNN
+F 0 "C35" H 1450 1350 50  0000 C CNN
+F 1 "10u" H 1450 1450 50  0000 C CNN
 F 2 "Capacitor_Tantalum_SMD:CP_EIA-3216-18_Kemet-A" H 1388 1100 50  0001 C CNN
 F 3 "~" H 1350 1250 50  0001 C CNN
@@
 	1350 1000 1550 1000
 Connection ~ 1550 1000
-$Comp
-L power:+9V #PWR032
-U 1 1 5C913F7B
-P 2800 1000
-F 0 "#PWR032" H 2800 850 50  0001 C CNN
-F 1 "+9V" H 2815 1173 50  0000 C CNN
-F 2 "" H 2800 1000 50  0001 C CNN
-F 3 "" H 2800 1000 50  0001 C CNN
-	1    2800 1000
-	0    1    1    0
-$EndComp
 Wire Wire Line
 	2800 1000 2700 1000
 Connection ~ 2700 1000
-$Comp
-L power:-9V #PWR027
-U 1 1 5C91410A
-P 1250 1000
-F 0 "#PWR027" H 1250 875 50  0001 C CNN
-F 1 "-9V" H 1265 1173 50  0000 C CNN
-F 2 "" H 1250 1000 50  0001 C CNN
-F 3 "" H 1250 1000 50  0001 C CNN
-	1    1250 1000
-	0    -1   -1   0
-$EndComp
 Wire Wire Line
 	1250 1000 1350 1000
@@
 P 3950 6250
 F 0 "U9" H 3950 6617 50  0000 C CNN
-F 1 "AD8620" H 3950 6526 50  0000 C CNN
+F 1 "AD8620/AD712" H 3950 6526 50  0000 C CNN
 F 2 "Housings_SOIC:SOIC-8_3.9x4.9mm_Pitch1.27mm" H 3950 6250 50  0001 C CNN
 F 3 "http://www.analog.com/media/en/technical-documentation/data-sheets/AD8610_8620.pdf" H 3950 6250 50  0001 C CNN
@@
 	0    1    1    0
 $EndComp
-$Comp
-L power:+9V #PWR037
-U 1 1 5CD91CF9
-P 7600 2450
-F 0 "#PWR037" H 7600 2300 50  0001 C CNN
-F 1 "+9V" H 7615 2623 50  0000 C CNN
-F 2 "" H 7600 2450 50  0001 C CNN
-F 3 "" H 7600 2450 50  0001 C CNN
-	1    7600 2450
-	1    0    0    -1
-$EndComp
 Wire Wire Line
 	7800 3350 7600 3350
@@
 Wire Wire Line
 	9250 3000 9150 3000
-$Comp
-L power:-9V #PWR040
-U 1 1 5CDCF6C9
-P 9150 2450
-F 0 "#PWR040" H 9150 2325 50  0001 C CNN
-F 1 "-9V" H 9165 2623 50  0000 C CNN
-F 2 "" H 9150 2450 50  0001 C CNN
-F 3 "" H 9150 2450 50  0001 C CNN
-	1    9150 2450
-	1    0    0    -1
-$EndComp
 Connection ~ 9150 3000
 Wire Wire Line
@@
 Wire Wire Line
 	8500 1650 8500 1500
+$Comp
+L power:-12V #PWR?
+U 1 1 5E6E09BC
+P 1250 1000
+F 0 "#PWR?" H 1250 1100 50  0001 C CNN
+F 1 "-12V" V 1265 1128 50  0000 L CNN
+F 2 "" H 1250 1000 50  0001 C CNN
+F 3 "" H 1250 1000 50  0001 C CNN
+	1    1250 1000
+	0    -1   -1   0
+$EndComp
+$Comp
+L power:+12V #PWR?
+U 1 1 5E6E1025
+P 2800 1000
+F 0 "#PWR?" H 2800 850 50  0001 C CNN
+F 1 "+12V" V 2815 1128 50  0000 L CNN
+F 2 "" H 2800 1000 50  0001 C CNN
+F 3 "" H 2800 1000 50  0001 C CNN
+	1    2800 1000
+	0    1    1    0
+$EndComp
+$Comp
+L power:+12V #PWR?
+U 1 1 5E70368A
+P 7600 2450
+F 0 "#PWR?" H 7600 2300 50  0001 C CNN
+F 1 "+12V" H 7615 2623 50  0000 C CNN
+F 2 "" H 7600 2450 50  0001 C CNN
+F 3 "" H 7600 2450 50  0001 C CNN
+	1    7600 2450
+	1    0    0    -1
+$EndComp
+$Comp
+L power:-12V #PWR?
+U 1 1 5E709A61
+P 9150 2450
+F 0 "#PWR?" H 9150 2550 50  0001 C CNN
+F 1 "-12V" H 9165 2623 50  0000 C CNN
+F 2 "" H 9150 2450 50  0001 C CNN
+F 3 "" H 9150 2450 50  0001 C CNN
+	1    9150 2450
+	1    0    0    -1
+$EndComp
 $EndSCHEMATC

Commit message: minor changes & pdf update
Parts:
- TP1: value TestPoint -> SolderingHole
Other:
- moved on the sheet: TP1
Changed lines of the file:
@@
 L Connector:TestPoint TP1
 U 1 1 5E58C58D
-P 8500 1500
-F 0 "TP1" H 8558 1618 50  0000 L CNN
-F 1 "TestPoint" H 8558 1527 50  0000 L CNN
-F 2 "TestPoint:TestPoint_Plated_Hole_D2.0mm" H 8700 1500 50  0001 C CNN
-F 3 "~" H 8700 1500 50  0001 C CNN
-	1    8500 1500
+P 8350 1350
+F 0 "TP1" H 8408 1468 50  0000 L CNN
+F 1 "SolderingHole" H 8408 1377 50  0000 L CNN
+F 2 "TestPoint:TestPoint_Plated_Hole_D2.0mm" H 8550 1350 50  0001 C CNN
+F 3 "~" H 8550 1350 50  0001 C CNN
+	1    8350 1350
 	1    0    0    -1
 $EndComp
@@
 L power:GND #PWR062
 U 1 1 5E58D3F2
-P 8500 1650
-F 0 "#PWR062" H 8500 1400 50  0001 C CNN
-F 1 "GND" H 8505 1477 50  0000 C CNN
-F 2 "" H 8500 1650 50  0001 C CNN
-F 3 "" H 8500 1650 50  0001 C CNN
-	1    8500 1650
+P 8350 1500
+F 0 "#PWR062" H 8350 1250 50  0001 C CNN
+F 1 "GND" H 8355 1327 50  0000 C CNN
+F 2 "" H 8350 1500 50  0001 C CNN
+F 3 "" H 8350 1500 50  0001 C CNN
+	1    8350 1500
 	1    0    0    -1
 $EndComp
 Wire Wire Line
-	8500 1650 8500 1500
+	8350 1500 8350 1350
 $Comp
 L power:-12V #PWR0107

Commit message: new pdf and minor changes in schematics and fw
Parts:
- U9: value AD8620/AD712 -> AD8066
Changed lines of the file:
@@
 P 3850 3550
 F 0 "U9" H 3850 3917 50  0000 C CNN
-F 1 "AD8620/AD712" H 3850 3826 50  0000 C CNN
+F 1 "AD8066" H 3850 3826 50  0000 C CNN
 F 2 "Housings_SOIC:SOIC-8_3.9x4.9mm_Pitch1.27mm" H 3850 3550 50  0001 C CNN
 F 3 "http://www.analog.com/media/en/technical-documentation/data-sheets/AD8610_8620.pdf" H 3850 3550 50  0001 C CNN
@@
 P 2000 1100
 F 0 "U9" V 2100 1100 50  0000 L CNN
-F 1 "AD8620/AD712" V 2000 850 50  0000 L CNN
+F 1 "AD8066" V 2000 950 50  0000 L CNN
 F 2 "Housings_SOIC:SOIC-8_3.9x4.9mm_Pitch1.27mm" H 2000 1100 50  0001 C CNN
 F 3 "http://www.analog.com/media/en/technical-documentation/data-sheets/AD8610_8620.pdf" H 2000 1100 50  0001 C CNN
@@
 P 3950 6250
 F 0 "U9" H 3950 6617 50  0000 C CNN
-F 1 "AD8620/AD712" H 3950 6526 50  0000 C CNN
+F 1 "AD8066" H 3950 6526 50  0000 C CNN
 F 2 "Housings_SOIC:SOIC-8_3.9x4.9mm_Pitch1.27mm" H 3950 6250 50  0001 C CNN
 F 3 "http://www.analog.com/media/en/technical-documentation/data-sheets/AD8610_8620.pdf" H 3950 6250 50  0001 C CNN
