File: schematics/DykoDAC.sch (KiCad schematic (older format))
At the start: 0 parts

Commit message: finishing
Changed lines of the file:
@@
 $EndDescr
 $Sheet
-S 750  750  1200 1150
+S 750  750  1200 1300
 U 5C91BC19
 F0 "PowerSupply" 50
@@
 $EndSheet
 $Sheet
-S 2200 800  1300 1350
+S 2200 800  1300 1200
 U 5CF60BAD
 F0 "DykoDAC_MCU" 47
