File: schematics/DykoDAC_MCU.sch (KiCad schematic (older format))
At the start: 19 parts

Commit message: mcu input and usb added, oscilators moved to DAC schematics
Parts:
- removed C? (x2): 100n, symbol Device:C
- removed R? (x2): 22, symbol Device:R
- removed R? (x2): 10k, symbol Device:R
- removed X?: 22.5792Mhz, Oscillator:Oscillator_SMD_TXC_7C-4Pin_5.0x3.2mm, symbol Oscillator:TXC-7C
- removed X?: 24.576Mhz, Oscillator:Oscillator_SMD_TXC_7C-4Pin_5.0x3.2mm, symbol Oscillator:TXC-7C
- added C? (x3): 0.1u, symbol Device:C
- added J?: Conn_01x02_Male, symbol Connector:Conn_01x02_Male
- added J?: Debug, symbol Connector_Generic:Conn_02x04_Odd_Even
- added R?: 30k, symbol Device:R
- added R?: 47k, symbol Device:R
- added R? (x4): 10k, symbol Device:R
- added R? (x3): 22, symbol Device:R
- added SW?: PEC09-2120K, symbol Device:Rotary_Encoder_Switch
- C?: value C -> 0.1u
- C?: value 4.5n -> 1n
Connections:
- net labels added: +3V3, DBG_RX, DBG_TX, ENC_A, ENC_B, ENC_BUTTON, RST, SWCLK, SWDIO, S_DOUT, S_LRCK, S_SCLK, VBUS_3V3
- net labels removed: 3V3_OSC, OSC_EN_1, OSC_EN_2, S_MCLK, VBUS
- wire segments 88 -> 120
Other:
- moved on the sheet: C?, L?

Commit message: finishing
Parts:
- added D?: LED, symbol Device:LED
- added J4: OLED, Pin_Headers:Pin_Header_Angled_1x04_Pitch2.54mm, symbol Connector_Generic:Conn_01x04
- added R33, R34: 2k7, Resistors_SMD:R_1206, symbol Device:R
- added R?: 680, symbol Device:R
- C55, C56, C57, C58, C59, C60, C61, C62, C63: renamed from C?; footprint (none) -> Capacitors_SMD:C_1206
- J3: renamed from J?; footprint (none) -> Connect:USB_B
- J5: renamed from J?; footprint (none) -> Pin_Headers:Pin_Header_Straight_2x04_Pitch2.54mm
- J6: renamed from J?; footprint (none) -> Pin_Headers:Pin_Header_Straight_1x02_Pitch2.54mm
- L2: renamed from L?; footprint (none) -> Choke_SMD:Choke_SMD_1206_Standard
- R27, R28, R29, R30, R31, R32, R35, R36, R37, R38: renamed from R?; footprint (none) -> Resistors_SMD:R_1206
- SW1: renamed from SW?; footprint (none) -> Pin_Headers:Pin_Header_Angled_1x05_Pitch2.54mm
- U11: renamed from U?; footprint (none) -> Housings_SSOP:TSOP-6_1.65x3.05mm_Pitch0.95mm
- gave numbers to parts that had none: 1
Connections:
- net labels added: DAC_CS, DAC_RST, LED_TEST, MCU_MISO, MCU_MOSI, MCU_SCK, OLED_SCL, OLED_SDA, OSC_EN_1, OSC_EN_2
- wire segments 120 -> 147
- no-connect marks 0 -> 14
Other:
- moved on the sheet: C55, C56, C57, C58, C59, C60, C61, C62, C63, J3, L2, R27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

Commit message: changed filter values started with PCB design
Parts:
- D3: renamed from D?; footprint (none) -> LEDs:LED_1206
- R39: renamed from R?; footprint (none) -> Resistors_SMD:R_1206
- U12: footprint Package_QFP:TQFP-48_7x7mm_P0.5mm -> Housings_QFP:TQFP-48_7x7mm_Pitch0.5mm
Other:
- moved on the sheet: D3, R38, R39
Changed lines of the file:
@@
 F 0 "U12" H 9150 4000 50  0000 C CNN
 F 1 "ATSAMD21G18A-AUT" H 9150 3800 50  0000 C CNN
-F 2 "Package_QFP:TQFP-48_7x7mm_P0.5mm" H 8200 2150 50  0001 C CNN
+F 2 "Housings_QFP:TQFP-48_7x7mm_Pitch0.5mm" H 8200 2150 50  0001 C CNN
 F 3 "http://ww1.microchip.com/downloads/en/DeviceDoc/SAMD21-Family-DataSheet-DS40001882D.pdf" H 9150 4900 50  0001 C CNN
 	1    9150 3900
@@
 L Connector:Conn_01x02_Male J6
 U 1 1 5D133620
-P 5550 6900
-F 0 "J6" H 5600 7000 50  0000 C CNN
-F 1 "Conn_01x02_Male" H 5658 6990 50  0001 C CNN
-F 2 "Pin_Headers:Pin_Header_Straight_1x02_Pitch2.54mm" H 5550 6900 50  0001 C CNN
-F 3 "~" H 5550 6900 50  0001 C CNN
-	1    5550 6900
+P 3250 6500
+F 0 "J6" H 3300 6600 50  0000 C CNN
+F 1 "Conn_01x02_Male" H 3358 6590 50  0001 C CNN
+F 2 "Pin_Headers:Pin_Header_Straight_1x02_Pitch2.54mm" H 3250 6500 50  0001 C CNN
+F 3 "~" H 3250 6500 50  0001 C CNN
+	1    3250 6500
 	1    0    0    -1
 $EndComp
@@
 L power:GND #PWR065
 U 1 1 5D136B73
-P 5850 7100
-F 0 "#PWR065" H 5850 6850 50  0001 C CNN
-F 1 "GND" H 5855 6927 50  0000 C CNN
-F 2 "" H 5850 7100 50  0001 C CNN
-F 3 "" H 5850 7100 50  0001 C CNN
-	1    5850 7100
-	1    0    0    -1
-$EndComp
-Wire Wire Line
-	5750 7000 5850 7000
-Wire Wire Line
-	5850 7000 5850 7100
+P 3550 6700
+F 0 "#PWR065" H 3550 6450 50  0001 C CNN
+F 1 "GND" H 3555 6527 50  0000 C CNN
+F 2 "" H 3550 6700 50  0001 C CNN
+F 3 "" H 3550 6700 50  0001 C CNN
+	1    3550 6700
+	1    0    0    -1
+$EndComp
+Wire Wire Line
+	3450 6600 3550 6600
+Wire Wire Line
+	3550 6600 3550 6700
 $Comp
 L power:+3V3 #PWR064
 U 1 1 5D13B6EE
-P 5850 6400
-F 0 "#PWR064" H 5850 6250 50  0001 C CNN
-F 1 "+3V3" H 5865 6573 50  0000 C CNN
-F 2 "" H 5850 6400 50  0001 C CNN
-F 3 "" H 5850 6400 50  0001 C CNN
-	1    5850 6400
+P 3550 6000
+F 0 "#PWR064" H 3550 5850 50  0001 C CNN
+F 1 "+3V3" H 3565 6173 50  0000 C CNN
+F 2 "" H 3550 6000 50  0001 C CNN
+F 3 "" H 3550 6000 50  0001 C CNN
+	1    3550 6000
 	1    0    0    -1
 $EndComp
@@
 L Device:R R38
 U 1 1 5D13C7BB
-P 5850 6650
-F 0 "R38" H 5920 6696 50  0000 L CNN
-F 1 "10k" H 5920 6605 50  0000 L CNN
-F 2 "Resistors_SMD:R_1206" V 5780 6650 50  0001 C CNN
-F 3 "~" H 5850 6650 50  0001 C CNN
-	1    5850 6650
-	1    0    0    -1
-$EndComp
-Wire Wire Line
-	5850 6500 5850 6400
-Wire Wire Line
-	5850 6800 5850 6900
-Wire Wire Line
-	5850 6900 5750 6900
-Text Label 6050 6900 2    47   ~ 0
+P 3550 6250
+F 0 "R38" H 3620 6296 50  0000 L CNN
+F 1 "10k" H 3620 6205 50  0000 L CNN
+F 2 "Resistors_SMD:R_1206" V 3480 6250 50  0001 C CNN
+F 3 "~" H 3550 6250 50  0001 C CNN
+	1    3550 6250
+	1    0    0    -1
+$EndComp
+Wire Wire Line
+	3550 6100 3550 6000
+Wire Wire Line
+	3550 6400 3550 6500
+Wire Wire Line
+	3550 6500 3450 6500
+Text Label 3750 6500 2    47   ~ 0
 RST
 Wire Wire Line
-	6050 6900 5850 6900
-Connection ~ 5850 6900
+	3750 6500 3550 6500
+Connection ~ 3550 6500
 Text Label 7750 5400 0    47   ~ 0
 RST
@@
 	7750 3800 8150 3800
 $Comp
-L Device:LED D?
+L Device:LED D3
 U 1 1 5D27E6B2
-P 3800 6750
-F 0 "D?" V 3839 6633 50  0000 R CNN
-F 1 "LED" V 3748 6633 50  0000 R CNN
-F 2 "" H 3800 6750 50  0001 C CNN
-F 3 "~" H 3800 6750 50  0001 C CNN
-	1    3800 6750
+P 5500 6600
+F 0 "D3" V 5539 6483 50  0000 R CNN
+F 1 "LED" V 5448 6483 50  0000 R CNN
+F 2 "LEDs:LED_1206" H 5500 6600 50  0001 C CNN
+F 3 "~" H 5500 6600 50  0001 C CNN
+	1    5500 6600
 	0    -1   -1   0
 $EndComp
 $Comp
-L Device:R R?
+L Device:R R39
 U 1 1 5D27FAB2
-P 3800 6300
-F 0 "R?" H 3870 6346 50  0000 L CNN
-F 1 "680" H 3870 6255 50  0000 L CNN
-F 2 "" V 3730 6300 50  0001 C CNN
-F 3 "~" H 3800 6300 50  0001 C CNN
-	1    3800 6300
-	1    0    0    -1
-$EndComp
-Text Label 3350 5950 0    47   ~ 0
+P 5500 6150
+F 0 "R39" H 5570 6196 50  0000 L CNN
+F 1 "680" H 5570 6105 50  0000 L CNN
+F 2 "Resistors_SMD:R_1206" V 5430 6150 50  0001 C CNN
+F 3 "~" H 5500 6150 50  0001 C CNN
+	1    5500 6150
+	1    0    0    -1
+$EndComp
+Text Label 5050 5800 0    47   ~ 0
 LED_TEST
 Wire Wire Line
-	3350 5950 3800 5950
-Wire Wire Line
-	3800 5950 3800 6150
-Wire Wire Line
-	3800 6450 3800 6600
-$Comp
-L power:GND #PWR?
+	5050 5800 5500 5800
+Wire Wire Line
+	5500 5800 5500 6000
+Wire Wire Line
+	5500 6300 5500 6450
+$Comp
+L power:GND #PWR066
 U 1 1 5D29B849
-P 3800 7050
-F 0 "#PWR?" H 3800 6800 50  0001 C CNN
-F 1 "GND" H 3805 6877 50  0000 C CNN
-F 2 "" H 3800 7050 50  0001 C CNN
-F 3 "" H 3800 7050 50  0001 C CNN
-	1    3800 7050
-	1    0    0    -1
-$EndComp
-Wire Wire Line
-	3800 6900 3800 7050
+P 5500 6900
+F 0 "#PWR066" H 5500 6650 50  0001 C CNN
+F 1 "GND" H 5505 6727 50  0000 C CNN
+F 2 "" H 5500 6900 50  0001 C CNN
+F 3 "" H 5500 6900 50  0001 C CNN
+	1    5500 6900
+	1    0    0    -1
+$EndComp
+Wire Wire Line
+	5500 6750 5500 6900
 Text Label 10550 2700 2    47   ~ 0
 LED_TEST

Commit message: changed usb protection IC
Parts:
- removed U11: IP4234CZ6, Housings_SSOP:TSOP-6_1.65x3.05mm_Pitch0.95mm, symbol kamtar:IP4234CZ6
- added U11: PRTR5V0U2X.215, TO_SOT_Packages_SMD:SOT-143, symbol kamtar:PRTR5V0U2X.215
Other:
- moved on the sheet: R31, R32
Changed lines of the file:
@@
 	1    0    0    -1
 $EndComp
-Text Label 4850 1150 2    50   ~ 0
+Text Label 4050 1250 2    50   ~ 0
 VBUS_3V3
-Text Label 3900 1350 2    50   ~ 0
+Text Label 3000 1450 2    50   ~ 0
 USB_D+
-Text Label 3900 1450 2    50   ~ 0
+Text Label 3000 1550 2    50   ~ 0
 USB_D-
 $Comp
@@
 	1500 1950 1500 1900
 $Comp
-L kamtar:IP4234CZ6 U?
-U 1 1 5CFBCCD6
-P 2950 1400
-AR Path="/5C8D0112/5CFBCCD6" Ref="U?"  Part="1"
-AR Path="/5CF60BAD/5CFBCCD6" Ref="U11"  Part="1"
-F 0 "U11" H 2700 1050 79  0000 C CNN
-F 1 "IP4234CZ6" H 2900 950 79  0000 C CNN
-F 2 "Housings_SSOP:TSOP-6_1.65x3.05mm_Pitch0.95mm" H 2950 1400 236 0001 C CNN
-F 3 "" H 2950 1400 236 0001 C CNN
-	1    2950 1400
-	1    0    0    -1
-$EndComp
-$Comp
-L power:GND #PWR?
-U 1 1 5CFBCCE4
-P 3700 1650
-AR Path="/5C8D0112/5CFBCCE4" Ref="#PWR?"  Part="1"
-AR Path="/5CF60BAD/5CFBCCE4" Ref="#PWR052"  Part="1"
-F 0 "#PWR052" H 3700 1400 50  0001 C CNN
-F 1 "GND" H 3705 1477 50  0000 C CNN
-F 2 "" H 3700 1650 50  0001 C CNN
-F 3 "" H 3700 1650 50  0001 C CNN
-	1    3700 1650
-	1    0    0    -1
-$EndComp
-$Comp
 L Device:C C55
 U 1 1 5CFBCCEF
@@
 Wire Wire Line
 	1500 2500 1500 2400
-Wire Wire Line
-	1900 1450 2350 1450
-Wire Wire Line
-	1900 1550 2350 1550
-Wire Wire Line
-	2350 1150 2350 1250
-Wire Wire Line
-	1900 1250 2350 1250
-Connection ~ 2350 1250
-Wire Wire Line
-	2350 1250 2350 1350
-Wire Wire Line
-	3550 1350 3900 1350
-Wire Wire Line
-	3550 1450 3900 1450
-Wire Wire Line
-	3550 1550 3700 1550
-Wire Wire Line
-	3700 1550 3700 1650
 $Comp
 L Device:C C61
@@
 L Device:R R31
 U 1 1 5D0B7820
-P 4250 1150
-F 0 "R31" V 4043 1150 50  0000 C CNN
-F 1 "30k" V 4134 1150 50  0000 C CNN
-F 2 "Resistors_SMD:R_1206" V 4180 1150 50  0001 C CNN
-F 3 "~" H 4250 1150 50  0001 C CNN
-	1    4250 1150
+P 3450 1250
+F 0 "R31" V 3243 1250 50  0000 C CNN
+F 1 "30k" V 3334 1250 50  0000 C CNN
+F 2 "Resistors_SMD:R_1206" V 3380 1250 50  0001 C CNN
+F 3 "~" H 3450 1250 50  0001 C CNN
+	1    3450 1250
 	0    1    1    0
 $EndComp
 Wire Wire Line
-	2350 1150 4100 1150
-Wire Wire Line
-	4400 1150 4450 1150
+	3600 1250 3650 1250
 $Comp
 L Device:R R32
 U 1 1 5D0BD216
-P 4450 1500
-F 0 "R32" H 4520 1546 50  0000 L CNN
-F 1 "47k" H 4520 1455 50  0000 L CNN
-F 2 "Resistors_SMD:R_1206" V 4380 1500 50  0001 C CNN
-F 3 "~" H 4450 1500 50  0001 C CNN
-	1    4450 1500
+P 3650 1600
+F 0 "R32" H 3720 1646 50  0000 L CNN
+F 1 "47k" H 3720 1555 50  0000 L CNN
+F 2 "Resistors_SMD:R_1206" V 3580 1600 50  0001 C CNN
+F 3 "~" H 3650 1600 50  0001 C CNN
+	1    3650 1600
 	1    0    0    -1
 $EndComp
@@
 L power:GND #PWR054
 U 1 1 5D0BD903
-P 4450 1750
-F 0 "#PWR054" H 4450 1500 50  0001 C CNN
-F 1 "GND" H 4455 1577 50  0000 C CNN
-F 2 "" H 4450 1750 50  0001 C CNN
-F 3 "" H 4450 1750 50  0001 C CNN
-	1    4450 1750
-	1    0    0    -1
-$EndComp
-Wire Wire Line
-	4450 1750 4450 1650
-Wire Wire Line
-	4450 1350 4450 1150
-Connection ~ 4450 1150
-Wire Wire Line
-	4450 1150 4850 1150
+P 3650 1850
+F 0 "#PWR054" H 3650 1600 50  0001 C CNN
+F 1 "GND" H 3655 1677 50  0000 C CNN
+F 2 "" H 3650 1850 50  0001 C CNN
+F 3 "" H 3650 1850 50  0001 C CNN
+	1    3650 1850
+	1    0    0    -1
+$EndComp
+Wire Wire Line
+	3650 1850 3650 1750
+Wire Wire Line
+	3650 1450 3650 1250
+Connection ~ 3650 1250
+Wire Wire Line
+	3650 1250 4050 1250
 Text Label 7750 4600 0    47   ~ 0
 VBUS_3V3
@@
 NoConn ~ 10150 2900
 NoConn ~ 10150 2800
+Wire Wire Line
+	1900 1550 2400 1550
+Wire Wire Line
+	1900 1450 2250 1450
+Wire Wire Line
+	1900 1250 2550 1250
+$Comp
+L kamtar:PRTR5V0U2X.215 U11
+U 1 1 5D1D054C
+P 2300 2200
+F 0 "U11" H 2678 2302 47  0000 L CNN
+F 1 "PRTR5V0U2X.215" H 2678 2215 47  0000 L CNN
+F 2 "TO_SOT_Packages_SMD:SOT-143" H 2300 2200 47  0001 C CNN
+F 3 "" H 2300 2200 47  0001 C CNN
+	1    2300 2200
+	1    0    0    -1
+$EndComp
+Wire Wire Line
+	2250 1900 2250 1450
+Connection ~ 2250 1450
+Wire Wire Line
+	2250 1450 3000 1450
+Wire Wire Line
+	2400 1900 2400 1550
+Connection ~ 2400 1550
+Wire Wire Line
+	2400 1550 3000 1550
+Wire Wire Line
+	2550 1900 2550 1250
+Connection ~ 2550 1250
+Wire Wire Line
+	2550 1250 3300 1250
+$Comp
+L power:GND #PWR0104
+U 1 1 5D1E57FC
+P 2100 1800
+F 0 "#PWR0104" H 2100 1550 50  0001 C CNN
+F 1 "GND" H 2105 1627 50  0000 C CNN
+F 2 "" H 2100 1800 50  0001 C CNN
+F 3 "" H 2100 1800 50  0001 C CNN
+	1    2100 1800
+	-1   0    0    1
+$EndComp
+Wire Wire Line
+	2100 1900 2100 1800
 $EndSCHEMATC

Commit message: lots of stuf ....
Parts:
- C55, C56, C57, C58, C59, C60, C61, C62, C63: footprint Capacitors_SMD:C_1206 -> Capacitors_SMD:C_0603_HandSoldering
- D3: footprint LEDs:LED_1206 -> LEDs:LED_0805_HandSoldering
- R27, R28, R29, R30, R31, R32, R33, R34, R35, R36, R37, R38, R39: footprint Resistors_SMD:R_1206 -> Resistors_SMD:R_0603_HandSoldering
Changed lines of the file:
@@
 F 0 "C63" V 9650 2050 50  0000 C CNN
 F 1 "1u" V 9550 1800 50  0000 C CNN
-F 2 "Capacitors_SMD:C_1206" H 9638 1750 50  0001 C CNN
+F 2 "Capacitors_SMD:C_0603_HandSoldering" H 9638 1750 50  0001 C CNN
 F 3 "~" H 9600 1900 50  0001 C CNN
 	1    9600 1900
@@
 F 0 "C62" V 9550 1250 50  0000 C CNN
 F 1 "0.1u" V 9650 1550 50  0000 C CNN
-F 2 "Capacitors_SMD:C_1206" H 9638 1250 50  0001 C CNN
+F 2 "Capacitors_SMD:C_0603_HandSoldering" H 9638 1250 50  0001 C CNN
 F 3 "~" H 9600 1400 50  0001 C CNN
 	1    9600 1400
@@
 F 0 "R27" H 1450 2150 50  0000 R CNN
 F 1 "1M" H 1450 2050 50  0000 R CNN
-F 2 "Resistors_SMD:R_1206" V 1430 2100 50  0001 C CNN
+F 2 "Resistors_SMD:R_0603_HandSoldering" V 1430 2100 50  0001 C CNN
 F 3 "~" H 1500 2100 50  0001 C CNN
 	1    1500 2100
@@
 F 0 "C55" H 1050 2200 50  0000 L CNN
 F 1 "1n" H 1250 2000 50  0000 L CNN
-F 2 "Capacitors_SMD:C_1206" H 1238 1950 50  0001 C CNN
+F 2 "Capacitors_SMD:C_0603_HandSoldering" H 1238 1950 50  0001 C CNN
 F 3 "~" H 1200 2100 50  0001 C CNN
 	1    1200 2100
@@
 F 0 "C61" V 8450 2100 50  0000 C CNN
 F 1 "0.1u" V 8450 1800 50  0000 C CNN
-F 2 "Capacitors_SMD:C_1206" H 8538 1800 50  0001 C CNN
+F 2 "Capacitors_SMD:C_0603_HandSoldering" H 8538 1800 50  0001 C CNN
 F 3 "~" H 8500 1950 50  0001 C CNN
 	1    8500 1950
@@
 F 0 "C60" V 8550 1850 50  0000 C CNN
 F 1 "0.1u" V 8450 1550 50  0000 C CNN
-F 2 "Capacitors_SMD:C_1206" H 8538 1550 50  0001 C CNN
+F 2 "Capacitors_SMD:C_0603_HandSoldering" H 8538 1550 50  0001 C CNN
 F 3 "~" H 8500 1700 50  0001 C CNN
 	1    8500 1700
@@
 F 0 "C59" V 8450 1250 50  0000 C CNN
 F 1 "1u" V 8550 1500 50  0000 C CNN
-F 2 "Capacitors_SMD:C_1206" H 8538 1250 50  0001 C CNN
+F 2 "Capacitors_SMD:C_0603_HandSoldering" H 8538 1250 50  0001 C CNN
 F 3 "~" H 8500 1400 50  0001 C CNN
 	1    8500 1400
@@
 F 0 "R31" V 3243 1250 50  0000 C CNN
 F 1 "30k" V 3334 1250 50  0000 C CNN
-F 2 "Resistors_SMD:R_1206" V 3380 1250 50  0001 C CNN
+F 2 "Resistors_SMD:R_0603_HandSoldering" V 3380 1250 50  0001 C CNN
 F 3 "~" H 3450 1250 50  0001 C CNN
 	1    3450 1250
@@
 F 0 "R32" H 3720 1646 50  0000 L CNN
 F 1 "47k" H 3720 1555 50  0000 L CNN
-F 2 "Resistors_SMD:R_1206" V 3580 1600 50  0001 C CNN
+F 2 "Resistors_SMD:R_0603_HandSoldering" V 3580 1600 50  0001 C CNN
 F 3 "~" H 3650 1600 50  0001 C CNN
 	1    3650 1600
@@
 F 0 "R28" H 4720 3546 50  0000 L CNN
 F 1 "10k" H 4720 3455 50  0000 L CNN
-F 2 "Resistors_SMD:R_1206" V 4580 3500 50  0001 C CNN
+F 2 "Resistors_SMD:R_0603_HandSoldering" V 4580 3500 50  0001 C CNN
 F 3 "~" H 4650 3500 50  0001 C CNN
 	1    4650 3500
@@
 F 0 "R29" H 4450 4300 50  0000 L CNN
 F 1 "10k" H 4450 4200 50  0000 L CNN
-F 2 "Resistors_SMD:R_1206" V 4580 4250 50  0001 C CNN
+F 2 "Resistors_SMD:R_0603_HandSoldering" V 4580 4250 50  0001 C CNN
 F 3 "~" H 4650 4250 50  0001 C CNN
 	1    4650 4250
@@
 F 0 "R30" H 5670 3546 50  0000 L CNN
 F 1 "10k" H 5670 3455 50  0000 L CNN
-F 2 "Resistors_SMD:R_1206" V 5530 3500 50  0001 C CNN
+F 2 "Resistors_SMD:R_0603_HandSoldering" V 5530 3500 50  0001 C CNN
 F 3 "~" H 5600 3500 50  0001 C CNN
 	1    5600 3500
@@
 F 0 "R38" H 3620 6296 50  0000 L CNN
 F 1 "10k" H 3620 6205 50  0000 L CNN
-F 2 "Resistors_SMD:R_1206" V 3480 6250 50  0001 C CNN
+F 2 "Resistors_SMD:R_0603_HandSoldering" V 3480 6250 50  0001 C CNN
 F 3 "~" H 3550 6250 50  0001 C CNN
 	1    3550 6250
@@
 F 0 "R36" V 7850 3500 50  0000 C CNN
 F 1 "22" V 7900 3250 50  0000 C CNN
-F 2 "Resistors_SMD:R_1206" V 7830 3300 50  0001 C CNN
+F 2 "Resistors_SMD:R_0603_HandSoldering" V 7830 3300 50  0001 C CNN
 F 3 "~" H 7900 3300 50  0001 C CNN
 	1    7900 3300
@@
 F 0 "R37" V 7850 3600 50  0000 C CNN
 F 1 "22" V 7900 3350 50  0000 C CNN
-F 2 "Resistors_SMD:R_1206" V 7830 3400 50  0001 C CNN
+F 2 "Resistors_SMD:R_0603_HandSoldering" V 7830 3400 50  0001 C CNN
 F 3 "~" H 7900 3400 50  0001 C CNN
 	1    7900 3400
@@
 F 0 "R35" V 7800 2900 50  0000 C CNN
 F 1 "22" V 7900 2950 50  0000 C CNN
-F 2 "Resistors_SMD:R_1206" V 7830 3000 50  0001 C CNN
+F 2 "Resistors_SMD:R_0603_HandSoldering" V 7830 3000 50  0001 C CNN
 F 3 "~" H 7900 3000 50  0001 C CNN
 	1    7900 3000
 	0    1    1    0
 $EndComp
-Text GLabel 7650 3000 0    47   Input ~ 0
-S_DOUT
-Wire Wire Line
-	7650 3000 7750 3000
 Wire Wire Line
 	8150 3000 8050 3000
@@
 F 0 "C56" H 4100 3550 50  0000 L CNN
 F 1 "0.1u" H 4100 3450 50  0000 L CNN
-F 2 "Capacitors_SMD:C_1206" H 4388 3350 50  0001 C CNN
+F 2 "Capacitors_SMD:C_0603_HandSoldering" H 4388 3350 50  0001 C CNN
 F 3 "~" H 4350 3500 50  0001 C CNN
 	1    4350 3500
@@
 F 0 "C57" H 4100 4350 50  0000 L CNN
 F 1 "0.1u" H 4100 4250 50  0000 L CNN
-F 2 "Capacitors_SMD:C_1206" H 4388 4150 50  0001 C CNN
+F 2 "Capacitors_SMD:C_0603_HandSoldering" H 4388 4150 50  0001 C CNN
 F 3 "~" H 4350 4300 50  0001 C CNN
 	1    4350 4300
@@
 F 0 "C58" H 5200 3550 50  0000 L CNN
 F 1 "0.1u" H 5200 3450 50  0000 L CNN
-F 2 "Capacitors_SMD:C_1206" H 5488 3350 50  0001 C CNN
+F 2 "Capacitors_SMD:C_0603_HandSoldering" H 5488 3350 50  0001 C CNN
 F 3 "~" H 5450 3500 50  0001 C CNN
 	1    5450 3500
@@
 F 0 "R34" H 1820 6296 50  0000 L CNN
 F 1 "2k7" H 1820 6205 50  0000 L CNN
-F 2 "Resistors_SMD:R_1206" V 1680 6250 50  0001 C CNN
+F 2 "Resistors_SMD:R_0603_HandSoldering" V 1680 6250 50  0001 C CNN
 F 3 "~" H 1750 6250 50  0001 C CNN
 	1    1750 6250
@@
 F 0 "R33" H 1400 6300 50  0000 L CNN
 F 1 "2k7" H 1400 6200 50  0000 L CNN
-F 2 "Resistors_SMD:R_1206" V 1530 6250 50  0001 C CNN
+F 2 "Resistors_SMD:R_0603_HandSoldering" V 1530 6250 50  0001 C CNN
 F 3 "~" H 1600 6250 50  0001 C CNN
 	1    1600 6250
@@
 F 0 "D3" V 5539 6483 50  0000 R CNN
 F 1 "LED" V 5448 6483 50  0000 R CNN
-F 2 "LEDs:LED_1206" H 5500 6600 50  0001 C CNN
+F 2 "LEDs:LED_0805_HandSoldering" H 5500 6600 50  0001 C CNN
 F 3 "~" H 5500 6600 50  0001 C CNN
 	1    5500 6600
@@
 F 0 "R39" H 5570 6196 50  0000 L CNN
 F 1 "680" H 5570 6105 50  0000 L CNN
-F 2 "Resistors_SMD:R_1206" V 5430 6150 50  0001 C CNN
+F 2 "Resistors_SMD:R_0603_HandSoldering" V 5430 6150 50  0001 C CNN
 F 3 "~" H 5500 6150 50  0001 C CNN
 	1    5500 6150
@@
 Wire Wire Line
 	2100 1900 2100 1800
+Wire Wire Line
+	7650 3000 7750 3000
+Text GLabel 7650 3000 0    47   Input ~ 0
+S_DOUT
 $EndSCHEMATC
