File: schematics/DykoDAC_MCU.sch (KiCad schematic (older format))
At the start: 31 parts, among them J3 USB_B, J4 OLED, J5 Debug, J6 Conn_01x02_Male, SW1 PEC09-2120K, U11 PRTR5V0U2X.215, U12 ATSAMD21G18A-AUT

Commit message: no message
Parts:
- removed L2: 100u, Choke_SMD:Choke_SMD_1206_Standard, symbol Device:L
- C55, C56, C57, C58, C59, C60, C61, C62, C63: footprint Capacitors_SMD:C_0603_HandSoldering -> Capacitors_SMD:C_0603
- D3: footprint LEDs:LED_0805_HandSoldering -> LEDs:LED_D3.0mm
- R27, R28, R29, R30, R31, R32, R33, R34, R35, R36, R37, R38, R39: footprint Resistors_SMD:R_0603_HandSoldering -> Resistors_SMD:R_0603
Connections:
- wire segments 147 -> 146
Changed lines of the file:
@@
 EESchema Schematic File Version 4
-LIBS:DykoDAC-cache
-EELAYER 29 0
+EELAYER 30 0
 EELAYER END
 $Descr A4 11693 8268
@@
 F 0 "C63" V 9650 2050 50  0000 C CNN
 F 1 "1u" V 9550 1800 50  0000 C CNN
-F 2 "Capacitors_SMD:C_0603_HandSoldering" H 9638 1750 50  0001 C CNN
+F 2 "Capacitors_SMD:C_0603" H 9638 1750 50  0001 C CNN
 F 3 "~" H 9600 1900 50  0001 C CNN
 	1    9600 1900
@@
 	1    0    0    -1
 $EndComp
-$Comp
-L Device:L L2
-U 1 1 5CF8623C
-P 9050 1400
-F 0 "L2" V 9240 1400 50  0000 C CNN
-F 1 "100u" V 9149 1400 50  0000 C CNN
-F 2 "Choke_SMD:Choke_SMD_1206_Standard" H 9050 1400 50  0001 C CNN
-F 3 "~" H 9050 1400 50  0001 C CNN
-	1    9050 1400
-	0    -1   -1   0
-$EndComp
 Wire Wire Line
 	9250 2000 9250 1400
-Wire Wire Line
-	9250 1400 9200 1400
-Wire Wire Line
-	8900 1400 8800 1400
 Wire Wire Line
 	8800 1400 8800 1300
@@
 F 0 "C62" V 9550 1250 50  0000 C CNN
 F 1 "0.1u" V 9650 1550 50  0000 C CNN
-F 2 "Capacitors_SMD:C_0603_HandSoldering" H 9638 1250 50  0001 C CNN
+F 2 "Capacitors_SMD:C_0603" H 9638 1250 50  0001 C CNN
 F 3 "~" H 9600 1400 50  0001 C CNN
 	1    9600 1400
@@
 F 0 "R27" H 1450 2150 50  0000 R CNN
 F 1 "1M" H 1450 2050 50  0000 R CNN
-F 2 "Resistors_SMD:R_0603_HandSoldering" V 1430 2100 50  0001 C CNN
+F 2 "Resistors_SMD:R_0603" V 1430 2100 50  0001 C CNN
 F 3 "~" H 1500 2100 50  0001 C CNN
 	1    1500 2100
@@
 F 0 "C55" H 1050 2200 50  0000 L CNN
 F 1 "1n" H 1250 2000 50  0000 L CNN
-F 2 "Capacitors_SMD:C_0603_HandSoldering" H 1238 1950 50  0001 C CNN
+F 2 "Capacitors_SMD:C_0603" H 1238 1950 50  0001 C CNN
 F 3 "~" H 1200 2100 50  0001 C CNN
 	1    1200 2100
@@
 F 0 "C61" V 8450 2100 50  0000 C CNN
 F 1 "0.1u" V 8450 1800 50  0000 C CNN
-F 2 "Capacitors_SMD:C_0603_HandSoldering" H 8538 1800 50  0001 C CNN
+F 2 "Capacitors_SMD:C_0603" H 8538 1800 50  0001 C CNN
 F 3 "~" H 8500 1950 50  0001 C CNN
 	1    8500 1950
@@
 F 0 "C60" V 8550 1850 50  0000 C CNN
 F 1 "0.1u" V 8450 1550 50  0000 C CNN
-F 2 "Capacitors_SMD:C_0603_HandSoldering" H 8538 1550 50  0001 C CNN
+F 2 "Capacitors_SMD:C_0603" H 8538 1550 50  0001 C CNN
 F 3 "~" H 8500 1700 50  0001 C CNN
 	1    8500 1700
@@
 F 0 "C59" V 8450 1250 50  0000 C CNN
 F 1 "1u" V 8550 1500 50  0000 C CNN
-F 2 "Capacitors_SMD:C_0603_HandSoldering" H 8538 1250 50  0001 C CNN
+F 2 "Capacitors_SMD:C_0603" H 8538 1250 50  0001 C CNN
 F 3 "~" H 8500 1400 50  0001 C CNN
 	1    8500 1400
@@
 F 0 "R31" V 3243 1250 50  0000 C CNN
 F 1 "30k" V 3334 1250 50  0000 C CNN
-F 2 "Resistors_SMD:R_0603_HandSoldering" V 3380 1250 50  0001 C CNN
+F 2 "Resistors_SMD:R_0603" V 3380 1250 50  0001 C CNN
 F 3 "~" H 3450 1250 50  0001 C CNN
 	1    3450 1250
@@
 F 0 "R32" H 3720 1646 50  0000 L CNN
 F 1 "47k" H 3720 1555 50  0000 L CNN
-F 2 "Resistors_SMD:R_0603_HandSoldering" V 3580 1600 50  0001 C CNN
+F 2 "Resistors_SMD:R_0603" V 3580 1600 50  0001 C CNN
 F 3 "~" H 3650 1600 50  0001 C CNN
 	1    3650 1600
@@
 F 0 "R28" H 4720 3546 50  0000 L CNN
 F 1 "10k" H 4720 3455 50  0000 L CNN
-F 2 "Resistors_SMD:R_0603_HandSoldering" V 4580 3500 50  0001 C CNN
+F 2 "Resistors_SMD:R_0603" V 4580 3500 50  0001 C CNN
 F 3 "~" H 4650 3500 50  0001 C CNN
 	1    4650 3500
@@
 F 0 "R29" H 4450 4300 50  0000 L CNN
 F 1 "10k" H 4450 4200 50  0000 L CNN
-F 2 "Resistors_SMD:R_0603_HandSoldering" V 4580 4250 50  0001 C CNN
+F 2 "Resistors_SMD:R_0603" V 4580 4250 50  0001 C CNN
 F 3 "~" H 4650 4250 50  0001 C CNN
 	1    4650 4250
@@
 F 0 "R30" H 5670 3546 50  0000 L CNN
 F 1 "10k" H 5670 3455 50  0000 L CNN
-F 2 "Resistors_SMD:R_0603_HandSoldering" V 5530 3500 50  0001 C CNN
+F 2 "Resistors_SMD:R_0603" V 5530 3500 50  0001 C CNN
 F 3 "~" H 5600 3500 50  0001 C CNN
 	1    5600 3500
@@
 F 0 "R38" H 3620 6296 50  0000 L CNN
 F 1 "10k" H 3620 6205 50  0000 L CNN
-F 2 "Resistors_SMD:R_0603_HandSoldering" V 3480 6250 50  0001 C CNN
+F 2 "Resistors_SMD:R_0603" V 3480 6250 50  0001 C CNN
 F 3 "~" H 3550 6250 50  0001 C CNN
 	1    3550 6250
@@
 F 0 "R36" V 7850 3500 50  0000 C CNN
 F 1 "22" V 7900 3250 50  0000 C CNN
-F 2 "Resistors_SMD:R_0603_HandSoldering" V 7830 3300 50  0001 C CNN
+F 2 "Resistors_SMD:R_0603" V 7830 3300 50  0001 C CNN
 F 3 "~" H 7900 3300 50  0001 C CNN
 	1    7900 3300
@@
 F 0 "R37" V 7850 3600 50  0000 C CNN
 F 1 "22" V 7900 3350 50  0000 C CNN
-F 2 "Resistors_SMD:R_0603_HandSoldering" V 7830 3400 50  0001 C CNN
+F 2 "Resistors_SMD:R_0603" V 7830 3400 50  0001 C CNN
 F 3 "~" H 7900 3400 50  0001 C CNN
 	1    7900 3400
@@
 F 0 "R35" V 7800 2900 50  0000 C CNN
 F 1 "22" V 7900 2950 50  0000 C CNN
-F 2 "Resistors_SMD:R_0603_HandSoldering" V 7830 3000 50  0001 C CNN
+F 2 "Resistors_SMD:R_0603" V 7830 3000 50  0001 C CNN
 F 3 "~" H 7900 3000 50  0001 C CNN
 	1    7900 3000
@@
 F 0 "C56" H 4100 3550 50  0000 L CNN
 F 1 "0.1u" H 4100 3450 50  0000 L CNN
-F 2 "Capacitors_SMD:C_0603_HandSoldering" H 4388 3350 50  0001 C CNN
+F 2 "Capacitors_SMD:C_0603" H 4388 3350 50  0001 C CNN
 F 3 "~" H 4350 3500 50  0001 C CNN
 	1    4350 3500
@@
 F 0 "C57" H 4100 4350 50  0000 L CNN
 F 1 "0.1u" H 4100 4250 50  0000 L CNN
-F 2 "Capacitors_SMD:C_0603_HandSoldering" H 4388 4150 50  0001 C CNN
+F 2 "Capacitors_SMD:C_0603" H 4388 4150 50  0001 C CNN
 F 3 "~" H 4350 4300 50  0001 C CNN
 	1    4350 4300
@@
 F 0 "C58" H 5200 3550 50  0000 L CNN
 F 1 "0.1u" H 5200 3450 50  0000 L CNN
-F 2 "Capacitors_SMD:C_0603_HandSoldering" H 5488 3350 50  0001 C CNN
+F 2 "Capacitors_SMD:C_0603" H 5488 3350 50  0001 C CNN
 F 3 "~" H 5450 3500 50  0001 C CNN
 	1    5450 3500
@@
 F 0 "R34" H 1820 6296 50  0000 L CNN
 F 1 "2k7" H 1820 6205 50  0000 L CNN
-F 2 "Resistors_SMD:R_0603_HandSoldering" V 1680 6250 50  0001 C CNN
+F 2 "Resistors_SMD:R_0603" V 1680 6250 50  0001 C CNN
 F 3 "~" H 1750 6250 50  0001 C CNN
 	1    1750 6250
@@
 F 0 "R33" H 1400 6300 50  0000 L CNN
 F 1 "2k7" H 1400 6200 50  0000 L CNN
-F 2 "Resistors_SMD:R_0603_HandSoldering" V 1530 6250 50  0001 C CNN
+F 2 "Resistors_SMD:R_0603" V 1530 6250 50  0001 C CNN
 F 3 "~" H 1600 6250 50  0001 C CNN
 	1    1600 6250
@@
 F 0 "D3" V 5539 6483 50  0000 R CNN
 F 1 "LED" V 5448 6483 50  0000 R CNN
-F 2 "LEDs:LED_0805_HandSoldering" H 5500 6600 50  0001 C CNN
+F 2 "LEDs:LED_D3.0mm" H 5500 6600 50  0001 C CNN
 F 3 "~" H 5500 6600 50  0001 C CNN
 	1    5500 6600
@@
 F 0 "R39" H 5570 6196 50  0000 L CNN
 F 1 "680" H 5570 6105 50  0000 L CNN
-F 2 "Resistors_SMD:R_0603_HandSoldering" V 5430 6150 50  0001 C CNN
+F 2 "Resistors_SMD:R_0603" V 5430 6150 50  0001 C CNN
 F 3 "~" H 5500 6150 50  0001 C CNN
 	1    5500 6150
@@
 Text GLabel 7650 3000 0    47   Input ~ 0
 S_DOUT
+Wire Wire Line
+	8800 1400 9250 1400
 $EndSCHEMATC

Commit message: opamp filter pcb
Parts:
- removed C59: 1u, Capacitors_SMD:C_0603, symbol Device:C
- removed C63: 1u, Capacitors_SMD:C_0603, symbol Device:CP
- removed J5: Debug, Pin_Headers:Pin_Header_Straight_2x04_Pitch2.54mm, symbol Connector_Generic:Conn_02x04_Odd_Even
- removed J6: Conn_01x02_Male, Pin_Headers:Pin_Header_Straight_1x02_Pitch2.54mm, symbol Connector:Conn_01x02_Male
- added C59: 10u, Capacitors_Tantalum_SMD:CP_Tantalum_Case-A_EIA-3216-18_Reflow, symbol Device:CP
- added C63: 1u, Capacitors_SMD:C_0603, symbol Device:C
- added C66: 0.1u, Capacitors_SMD:C_0603, symbol Device:C
- added J5: Debug, Pin_Headers:Pin_Header_Angled_2x03_Pitch1.27mm, symbol Connector_Generic:Conn_02x03_Odd_Even
- added Q1: MMBT3904, TO_SOT_Packages_SMD:SOT-23, symbol Device:Q_NPN_BEC
- added R44: 50, Resistors_SMD:R_0603, symbol Device:R_Small
- added R45: 10k, Resistors_SMD:R_0603, symbol Device:R_Small
- R39: value 680 -> 240
- SW1: footprint Pin_Headers:Pin_Header_Angled_1x05_Pitch2.54mm -> Potentiometers:Potentiometer_Alps_RK097_Double_Vertical
Other:
- moved on the sheet: C56, C57, C58, D3, J4, R28, R29, R30, R33, R34, R38, R39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

Commit message: pcb update
Parts:
- added J6: ENC_CONN, Pin_Headers:Pin_Header_Straight_1x04_Pitch1.27mm, symbol Connector_Generic:Conn_01x04
- added J7, J9: Conn_01x03, Pin_Headers:Pin_Header_Straight_1x03_Pitch1.27mm, symbol Connector_Generic:Conn_01x03
- added J8: OLED, Pin_Headers:Pin_Header_Straight_1x04_Pitch1.27mm, symbol Connector_Generic:Conn_01x04
- J5: footprint Pin_Headers:Pin_Header_Angled_2x03_Pitch1.27mm -> Pin_Headers:Pin_Header_Straight_2x03_Pitch2.54mm
Connections:
- net labels added: 3V3_Conn, BTT
- wire segments 146 -> 163
Other:
- moved on the sheet: J4, R33, R34
