File: schematics/DykoDAC_MCU.sch (KiCad schematic (older format))
At the start: 37 parts, among them J3 USB_B, J4 OLED, J5 Debug, J6 ENC_CONN, J7 Conn_01x03, J8 OLED, J9 Conn_01x03, Q1 MMBT3904, SW1 PEC09-2120K, U11 PRTR5V0U2X.215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

Commit message: pcb
Parts:
- removed J6: ENC_CONN, Pin_Headers:Pin_Header_Straight_1x04_Pitch1.27mm, symbol Connector_Generic:Conn_01x04
- removed J7, J9: Conn_01x03, Pin_Headers:Pin_Header_Straight_1x03_Pitch1.27mm, symbol Connector_Generic:Conn_01x03
- removed J8: OLED, Pin_Headers:Pin_Header_Straight_1x04_Pitch1.27mm, symbol Connector_Generic:Conn_01x04
- removed Q1: MMBT3904, TO_SOT_Packages_SMD:SOT-23, symbol Device:Q_NPN_BEC
- removed R44: 50, Resistors_SMD:R_0603, symbol Device:R_Small
- removed R45: 10k, Resistors_SMD:R_0603, symbol Device:R_Small
- removed U12: ATSAMD21G18A-AUT, Housings_QFP:TQFP-48_7x7mm_Pitch0.5mm, symbol MCU_Microchip_SAMD:ATSAMD21G18A-AUT
- added C67: 3.3u, Capacitors_SMD:C_0805, symbol Device:C
- added C68: 0.1u, Capacitors_SMD:C_0603, symbol Device:C
- added J6, J8: Conn_01x05, Pin_Headers:Pin_Header_Straight_1x05_Pitch1.00mm, symbol Connector_Generic:Conn_01x05
- added J7, J9: Conn_01x04, Pin_Headers:Pin_Header_Straight_1x04_Pitch1.00mm, symbol Connector_Generic:Conn_01x04
- added L2: Ferrite Bead, Capacitors_SMD:C_0603, symbol Device:L
- added U13: ATSAMD51J20A-A, Housings_QFP:LQFP-64_10x10mm_Pitch0.5mm, symbol MCU_Microchip_SAMD:ATSAMD51J20A-A
- C63: value 1u -> 0.1u
- D3: footprint LEDs:LED_D3.0mm -> LEDs:LED_0603_HandSoldering
- R39: value 240 -> 1k
Connections:
- net labels added: 3V3_Oled, VDD_F
- net labels removed: +3.3V
- wire segments 163 -> 170
- no-connect marks 14 -> 1
Other:
- moved on the sheet: C59, C60, C61, C62, D3, R35, R36, R37, R39

Commit message: pcb
Parts:
- added R5: 1k, Resistors_SMD:R_0603, symbol Device:R
Connections:
- wire segments 170 -> 173
Changed lines of the file:
@@
 Wire Wire Line
 	8000 3050 7900 3050
-Text Label 7600 4650 0    47   ~ 0
+Text Label 6950 4650 0    47   ~ 0
 SWCLK
 Text Label 7600 4750 0    47   ~ 0
@@
 Wire Wire Line
 	7600 4750 8000 4750
-Wire Wire Line
-	8000 4650 7600 4650
 Text Label 7600 2050 0    47   ~ 0
 DBG_RX
@@
 Wire Wire Line
 	6200 5900 6800 5900
+$Comp
+L Device:R R5
+U 1 1 5E58D5F8
+P 7200 4450
+F 0 "R5" H 7270 4496 50  0000 L CNN
+F 1 "1k" H 7250 4400 50  0000 L CNN
+F 2 "Resistors_SMD:R_0603" V 7130 4450 50  0001 C CNN
+F 3 "~" H 7200 4450 50  0001 C CNN
+	1    7200 4450
+	1    0    0    -1
+$EndComp
+$Comp
+L power:+3V3 #PWR019
+U 1 1 5E58E516
+P 7200 4200
+F 0 "#PWR019" H 7200 4050 50  0001 C CNN
+F 1 "+3V3" H 7215 4373 50  0000 C CNN
+F 2 "" H 7200 4200 50  0001 C CNN
+F 3 "" H 7200 4200 50  0001 C CNN
+	1    7200 4200
+	1    0    0    -1
+$EndComp
+Wire Wire Line
+	7200 4300 7200 4200
+Wire Wire Line
+	6950 4650 7200 4650
+Wire Wire Line
+	7200 4600 7200 4650
+Connection ~ 7200 4650
+Wire Wire Line
+	7200 4650 8000 4650
 $EndSCHEMATC

Commit message: pcb
Parts:
- J6, J8: footprint Pin_Headers:Pin_Header_Straight_1x05_Pitch1.00mm -> Pin_Headers:Pin_Header_Straight_1x05_Pitch2.00mm
- J7, J9: footprint Pin_Headers:Pin_Header_Straight_1x04_Pitch1.00mm -> Pin_Headers:Pin_Header_Straight_1x04_Pitch2.00mm
Changed lines of the file:
@@
 F 0 "J6" H 5230 2492 50  0000 L CNN
 F 1 "Conn_01x05" H 5230 2401 50  0000 L CNN
-F 2 "Pin_Headers:Pin_Header_Straight_1x05_Pitch1.00mm" H 5150 2450 50  0001 C CNN
+F 2 "Pin_Headers:Pin_Header_Straight_1x05_Pitch2.00mm" H 5150 2450 50  0001 C CNN
 F 3 "~" H 5150 2450 50  0001 C CNN
 	1    5150 2450
@@
 F 0 "J8" H 2918 4267 50  0000 C CNN
 F 1 "Conn_01x05" H 2918 4176 50  0000 C CNN
-F 2 "Pin_Headers:Pin_Header_Straight_1x05_Pitch1.00mm" H 3000 3850 50  0001 C CNN
+F 2 "Pin_Headers:Pin_Header_Straight_1x05_Pitch2.00mm" H 3000 3850 50  0001 C CNN
 F 3 "~" H 3000 3850 50  0001 C CNN
 	1    3000 3850
@@
 F 0 "J7" H 2180 3192 50  0000 L CNN
 F 1 "Conn_01x04" H 2180 3101 50  0000 L CNN
-F 2 "Pin_Headers:Pin_Header_Straight_1x04_Pitch1.00mm" H 2100 3200 50  0001 C CNN
+F 2 "Pin_Headers:Pin_Header_Straight_1x04_Pitch2.00mm" H 2100 3200 50  0001 C CNN
 F 3 "~" H 2100 3200 50  0001 C CNN
 	1    2100 3200
@@
 F 0 "J9" H 1118 5067 50  0000 C CNN
 F 1 "Conn_01x04" H 1118 4976 50  0000 C CNN
-F 2 "Pin_Headers:Pin_Header_Straight_1x04_Pitch1.00mm" H 1200 4750 50  0001 C CNN
+F 2 "Pin_Headers:Pin_Header_Straight_1x04_Pitch2.00mm" H 1200 4750 50  0001 C CNN
 F 3 "~" H 1200 4750 50  0001 C CNN
 	1    1200 4750
