File: schematics/DykoDAC.kicad_pcb (KiCad board)
At the start: 2 copper layers, 159.8 x 100.1 mm, 140 parts, among them J1 AC Input, J2 AudioJack, J3 USB_B, J4 OLED, J5 Debug, J6 Conn_01x05, J7 Conn_01x04, J8 Conn_01x05, J9 Conn_01x04, SW1 PEC09-2120K, U1 LT1762-5, U10 TPA6120A2, U11 PRTR5V0U2X.215, U13 ATSAMD51J20A-A, U2 LM317, U3 LM337, U4 L7805, U5 78L05, U6 LP5907-3.3, U7 LP5907-3.3, U8 CS4398, U9 AD8620, X1 22.5792Mhz, X2 24.576Mhz

Commit message: pcb update
Parts:
- moved J8 106.0 mm to (132.2, 54.4)
- moved J9 42.7 mm to (138.7, 126.2)
- moved J4 4.35 mm to (144.8, 124.0)
- moved R21 0.57 mm to (123.4, 110.2)
- moved R24 0.57 mm to (123.4, 108.7)
- moved R22 0.25 mm to (138.2, 109.9)
- moved R23 0.25 mm to (138.2, 108.3)
- moved C48 0.25 mm to (138.3, 105.8)
- moved C9 0.18 mm to (107.8, 118.9)
Routing:
- net +3V3: track 187.6 -> 173.6 mm, vias 5 -> 7
- net +5VA: track 30.4 -> 41.7 mm, vias 2 -> 0
- net -9V: track 81.2 -> 88.1 mm
- net GND: track 100.0 -> 105.0 mm, vias 66 -> 97
- net +9V: track 102.6 -> 107.4 mm, vias 4 -> 6
- net /DykoDAC_CS4398/S_MCLK: track 6.69 -> 8.33 mm
- net Net-(J2-Pad3): track 30.1 -> 31.7 mm
- net Net-(R22-Pad1): track 4.00 -> 5.45 mm
- net Net-(C40-Pad1): track 4.39 -> 5.40 mm
- net Net-(C30-Pad1): track 5.79 -> 4.84 mm
- net Net-(R20-Pad1): track 24.6 -> 25.1 mm
- net (no net): vias 0 -> 27
- removed copper zone on F.Cu, net GND
Other:
- board size 159.8 x 100.1 mm -> 99.4 x 100.1 mm
