File: schematics/DykoDAC.kicad_pcb (KiCad board)
At the start: 2 copper layers, 99.4 x 100.1 mm, 140 parts, among them J1 AC Input, J2 AudioJack, J3 USB_B, J4 OLED, J5 Debug, J6 Conn_01x05, J7 Conn_01x04, J8 Conn_01x05, J9 Conn_01x04, SW1 PEC09-2120K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

Commit message: pcb
Parts:
- removed R6: 10k, Resistors_SMD:R_0603
- added TP1: TestPoint, Connect:1pin, F.Cu at (130.8, 108.8)
- J1: footprint Connect:BARREL_JACK -> Terminal_Blocks:TerminalBlock_Altech_AK300-2_P5.00mm
- R5: value 10k -> 1k
- moved R30 129.1 mm to (135.0, 58.5), turned to 90 degrees
- moved C57 123.3 mm to (131.6, 55.4), turned to 90 degrees
- moved C56 121.3 mm to (135.3, 51.3), turned to 90 degrees
- moved R33 119.0 mm to (141.7, 126.9), turned to 90 degrees
- moved C58 118.2 mm to (133.0, 58.4), turned to 90 degrees
- moved R28 117.1 mm to (130.2, 61.5)
- moved R34 113.3 mm to (141.0, 129.9), turned to 90 degrees
- moved R29 107.1 mm to (135.1, 55.2), turned to 90 degrees
- moved R5 49.7 mm to (70.4, 135.1), turned to 90 degrees
- moved C55 27.2 mm to (54.6, 108.8)
- moved R27 21.5 mm to (54.6, 110.4)
- moved C2 4.95 mm to (78.0, 70.7)
- moved C3 4.83 mm to (78.4, 53.1)
- moved J8 4.45 mm to (127.8, 54.5)
- moved J1 2.72 mm to (54.0, 55.5), turned to 270 degrees
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Connections:
- R5 pad 2: DAC_CS -> /DykoDAC_MCU/SWCLK
Routing:
- net Net-(D1-Pad2): track 21.2 -> 2.63 mm
- net VS_POS: track 68.1 -> 85.2 mm
- net Net-(C55-Pad1): track 0.00 -> 17.1 mm
- net VS_NEG: track 75.1 -> 61.0 mm
- net /DykoDAC_MCU/VDD_F: track 26.1 -> 34.3 mm, vias 0 -> 2
- net GND: track 105.0 -> 108.9 mm, vias 97 -> 260
- net Net-(F1-Pad2): track 6.18 -> 9.72 mm
- net /DykoDAC_MCU/SWCLK: track 19.2 -> 21.9 mm
- net +3V3: track 173.6 -> 175.4 mm, vias 7 -> 9
- net (no net): vias 27 -> 0
- added copper zone on F.Cu, net GND
- added copper zone on F.Cu, net Net-(D1-Pad2)
- added copper zone on F.Cu, net VS_NEG
- added copper zone on F.Cu, net VS_POS
- removed copper zone on F.Cu, net Net-(C38-Pad1)
Other:
- board text added: "15V 1A AC"
- board text added: "DykoDAC"

Commit message: pcb
Parts:
- J6, J8: footprint Pin_Headers:Pin_Header_Straight_1x05_Pitch1.00mm -> Pin_Headers:Pin_Header_Straight_1x05_Pitch2.00mm
- J7, J9: footprint Pin_Headers:Pin_Header_Straight_1x04_Pitch1.00mm -> Pin_Headers:Pin_Header_Straight_1x04_Pitch2.00mm
- moved J7 7.49 mm to (61.1, 100.3)
- moved R34 5.12 mm to (141.6, 124.8), turned to 270 degrees
- moved J6 4.94 mm to (85.1, 132.1)
- moved J9 4.75 mm to (137.0, 121.9)
- moved R33 4.55 mm to (139.4, 122.9), turned to 270 degrees
- moved J4 3.43 mm to (144.7, 127.4), turned to 180 degrees
- moved C2 0.28 mm to (78.2, 70.9)
Routing:
- net /DykoDAC_MCU/3V3_Oled: track 0.00 -> 10.5 mm
- net Net-(J4-Pad1): track 0.00 -> 9.35 mm
- net Net-(J4-Pad2): track 0.00 -> 9.12 mm, vias 0 -> 1
- net /DykoDAC_MCU/OLED_SDA: track 15.7 -> 23.3 mm
- net /DykoDAC_MCU/OLED_SCL: track 14.7 -> 21.9 mm
- net /DykoDAC_MCU/ENC_A: track 11.0 -> 14.9 mm
- net /DykoDAC_MCU/ENC_B: track 10.8 -> 13.8 mm
- net /DykoDAC_MCU/ENC_BUTTON: track 10.6 -> 12.8 mm
- net +3V3: track 175.4 -> 173.8 mm
- net GND: vias 260 -> 327

Commit message: pcb
Parts:
- J4: footprint Pin_Headers:Pin_Header_Angled_1x04_Pitch2.54mm -> Pin_Headers:Pin_Header_Straight_1x04_Pitch2.54mm
- X1, X2: footprint Oscillators:Oscillator_SMD_Abracon_ASE-4pin_3.2x2.5mm -> Oscillators:Oscillator_SMD_SeikoEpson_SG210-4pin_2.5x2.0mm_HandSoldering
- moved D1 5.23 mm to (67.7, 71.0)
- moved D2 5.21 mm to (67.3, 53.6)
- moved F1 4.96 mm to (66.7, 61.8)
- moved C2 3.56 mm to (78.2, 74.4)
- moved C3 2.92 mm to (78.2, 56.0)
- moved R34 1.53 mm to (140.1, 125.0)
- moved J4 1.53 mm to (143.1, 127.5)
- moved J9 1.53 mm to (135.5, 122.0)
- moved R33 1.53 mm to (137.9, 123.1)
- moved J2 0.38 mm to (141.2, 84.2)
- moved R1 0.13 mm to (90.3, 113.3)
Routing:
- net VS_NEG: track 61.0 -> 14.5 mm
- net VS_POS: track 85.2 -> 56.5 mm
- net Net-(F1-Pad2): track 9.72 -> 14.1 mm
- net Net-(D1-Pad2): track 2.63 -> 0.00 mm
- net -9V: track 88.1 -> 89.9 mm
- net GND: track 108.9 -> 110.0 mm, vias 327 -> 526
- net OSC_EN_2: track 17.0 -> 17.5 mm

Commit message: pcb update
Parts:
- U2, U3, U4: footprint TO_SOT_Packages_SMD:SOT-223-3_TabPin2 -> TO_SOT_Packages_SMD:TO-263-2
- moved C14 11.0 mm to (62.9, 92.2), turned to 180 degrees
- moved C12 9.40 mm to (60.7, 83.8)
- moved C17 9.01 mm to (61.6, 89.7), turned to 180 degrees
- moved C64 7.94 mm to (84.5, 97.8)
- moved C4 7.19 mm to (84.3, 92.6), turned to 270 degrees
- moved C8 6.87 mm to (122.3, 90.3)
- moved R41 6.73 mm to (88.4, 100.8), turned to 270 degrees
- moved R40 5.72 mm to (91.2, 100.1)
- moved C10 5.66 mm to (94.7, 99.9)
- moved U4 5.46 mm to (69.8, 85.6)
- moved C18 5.46 mm to (67.7, 92.8)
- moved C20 5.46 mm to (67.8, 98.4)
- moved U6 5.46 mm to (67.8, 95.8)
- moved C49 5.39 mm to (74.4, 96.1)
- moved C11 5.31 mm to (117.3, 97.3)
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Routing:
- net VS_POS: track 56.5 -> 19.4 mm, vias 0 -> 4
- net VS_NEG: track 14.5 -> 0.00 mm
- net -9V: track 89.9 -> 85.1 mm
- net GND: track 110.0 -> 105.5 mm, vias 526 -> 607
- net +3V3: track 173.8 -> 169.8 mm
- net Net-(C65-Pad2): track 8.18 -> 11.2 mm
- net Net-(C64-Pad1): track 7.64 -> 10.6 mm
- net +9V: track 107.8 -> 110.1 mm, vias 6 -> 11
- net Net-(J2-Pad3): track 31.3 -> 33.5 mm, vias 2 -> 4
- net (no net): track 0.00 -> 0.40 mm, vias 0 -> 1
- added copper zone on F.Cu, net Net-(C14-Pad1)

Commit message: no message
Routing:
- net -9V: track 85.1 -> 93.3 mm, vias 2 -> 6
- net +9V: track 110.1 -> 111.8 mm, vias 11 -> 16
- net GND: track 105.5 -> 105.9 mm, vias 607 -> 608
- net (no net): track 0.40 -> 0.00 mm, vias 1 -> 0
- added copper zone on B.Cu, net +9V

Commit message: no message
Routing:
- net GND: vias 608 -> 593
Changed lines of the file:
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@@
     (thickness 1.6)
     (drawings 14)
-    (tracks 1555)
+    (tracks 1540)
     (zones 0)
     (modules 140)
@@
   )
   (setup
-    (last_trace_width 1.48)
+    (last_trace_width 0.25)
     (user_trace_width 0.6)
     (user_trace_width 1.48)
@@
   (segment (start 104.902 120.0785) (end 104.902 120.0785) (width 0.6) (layer F.Cu) (net 1))
   (via (at 104.902 120.0785) (size 0.6) (drill 0.3) (layers F.Cu B.Cu) (net 1))
-  (via (at 70.9295 90.424) (size 0.6) (drill 0.3) (layers F.Cu B.Cu) (net 1))
+  (via (at 70.0024 91.2876) (size 0.6) (drill 0.3) (layers F.Cu B.Cu) (net 1))
   (via (at 73.279 90.3605) (size 0.6) (drill 0.3) (layers F.Cu B.Cu) (net 1))
   (via (at 69.5325 80.7085) (size 0.6) (drill 0.3) (layers F.Cu B.Cu) (net 1))
@@
   (via (at 142.748 94.361) (size 0.6) (drill 0.3) (layers F.Cu B.Cu) (net 1))
   (via (at 145.161 115.951) (size 0.6) (drill 0.3) (layers F.Cu B.Cu) (net 1))
-  (via (at 137.541 118.364) (size 0.6) (drill 0.3) (layers F.Cu B.Cu) (net 1))
+  (via (at 136.8044 117.4496) (size 0.6) (drill 0.3) (layers F.Cu B.Cu) (net 1))
   (via (at 132.207 132.207) (size 0.6) (drill 0.3) (layers F.Cu B.Cu) (net 1))
   (via (at 144.907 136.398) (size 0.6) (drill 0.3) (layers F.Cu B.Cu) (net 1))
@@
   (via (at 120.904 98.806) (size 0.6) (drill 0.3) (layers F.Cu B.Cu) (net 1))
   (via (at 127.635 98.933) (size 0.6) (drill 0.3) (layers F.Cu B.Cu) (net 1))
-  (via (at 128.778 97.663) (size 0.6) (drill 0.3) (layers F.Cu B.Cu) (net 1))
-  (via (at 130.683 95.758) (size 0.6) (drill 0.3) (layers F.Cu B.Cu) (net 1))
+  (via (at 129.3876 96.4184) (size 0.6) (drill 0.3) (layers F.Cu B.Cu) (net 1))
   (via (at 131.953 93.599) (size 0.6) (drill 0.3) (layers F.Cu B.Cu) (net 1))
-  (via (at 132.334 90.932) (size 0.6) (drill 0.3) (layers F.Cu B.Cu) (net 1))
-  (via (at 133.223 88.9) (size 0.6) (drill 0.3) (layers F.Cu B.Cu) (net 1))
-  (via (at 134.874 87.63) (size 0.6) (drill 0.3) (layers F.Cu B.Cu) (net 1))
-  (via (at 137.414 87.503) (size 0.6) (drill 0.3) (layers F.Cu B.Cu) (net 1))
-  (via (at 139.573 87.63) (size 0.6) (drill 0.3) (layers F.Cu B.Cu) (net 1))
-  (via (at 142.113 87.63) (size 0.6) (drill 0.3) (layers F.Cu B.Cu) (net 1))
+  (via (at 132.6388 90.0176) (size 0.6) (drill 0.3) (layers F.Cu B.Cu) (net 1))
+  (via (at 135.636 87.5792) (size 0.6) (drill 0.3) (layers F.Cu B.Cu) (net 1))
+  (via (at 140.6652 87.3252) (size 0.6) (drill 0.3) (layers F.Cu B.Cu) (net 1))
   (via (at 143.51 86.614) (size 0.6) (drill 0.3) (layers F.Cu B.Cu) (net 1))
-  (via (at 145.669 85.979) (size 0.6) (drill 0.3) (layers F.Cu B.Cu) (net 1))
+  (via (at 145.5928 84.3788) (size 0.6) (drill 0.3) (layers F.Cu B.Cu) (net 1))
   (via (at 129.667 99.695) (size 0.6) (drill 0.3) (layers F.Cu B.Cu) (net 1))
-  (via (at 130.81 98.806) (size 0.6) (drill 0.3) (layers F.Cu B.Cu) (net 1))
-  (via (at 132.334 97.409) (size 0.6) (drill 0.3) (layers F.Cu B.Cu) (net 1))
-  (via (at 133.604 96.012) (size 0.6) (drill 0.3) (layers F.Cu B.Cu) (net 1))
-  (via (at 134.366 94.996) (size 0.6) (drill 0.3) (layers F.Cu B.Cu) (net 1))
+  (via (at 131.7244 97.6884) (size 0.6) (drill 0.3) (layers F.Cu B.Cu) (net 1))
+  (via (at 134.112 95.25) (size 0.6) (drill 0.3) (layers F.Cu B.Cu) (net 1))
   (via (at 134.747 92.71) (size 0.6) (drill 0.3) (layers F.Cu B.Cu) (net 1))
-  (via (at 134.874 91.186) (size 0.6) (drill 0.3) (layers F.Cu B.Cu) (net 1))
-  (via (at 136.017 90.17) (size 0.6) (drill 0.3) (layers F.Cu B.Cu) (net 1))
+  (via (at 135.3312 90.2716) (size 0.6) (drill 0.3) (layers F.Cu B.Cu) (net 1))
   (via (at 136.398 96.139) (size 0.6) (drill 0.3) (layers F.Cu B.Cu) (net 1))
-  (via (at 137.287 97.155) (size 0.6) (drill 0.3) (layers F.Cu B.Cu) (net 1))
   (via (at 138.43 98.298) (size 0.6) (drill 0.3) (layers F.Cu B.Cu) (net 1))
-  (via (at 138.811 99.441) (size 0.6) (drill 0.3) (layers F.Cu B.Cu) (net 1))
-  (via (at 139.0015 100.5205) (size 0.6) (drill 0.3) (layers F.Cu B.Cu) (net 1))
   (via (at 138.811 101.346) (size 0.6) (drill 0.3) (layers F.Cu B.Cu) (net 1))
   (via (at 132.969 99.695) (size 0.6) (drill 0.3) (layers F.Cu B.Cu) (net 1))
   (via (at 135.89 99.695) (size 0.6) (drill 0.3) (layers F.Cu B.Cu) (net 1))
   (via (at 135.001 97.917) (size 0.6) (drill 0.3) (layers F.Cu B.Cu) (net 1))
-  (via (at 140.208 105.283) (size 0.6) (drill 0.3) (layers F.Cu B.Cu) (net 1))
   (via (at 140.843 104.521) (size 0.6) (drill 0.3) (layers F.Cu B.Cu) (net 1))
-  (via (at 140.97 103.251) (size 0.6) (drill 0.3) (layers F.Cu B.Cu) (net 1))
   (via (at 141.097 101.6) (size 0.6) (drill 0.3) (layers F.Cu B.Cu) (net 1))
-  (via (at 141.224 100.33) (size 0.6) (drill 0.3) (layers F.Cu B.Cu) (net 1))
   (via (at 141.224 98.933) (size 0.6) (drill 0.3) (layers F.Cu B.Cu) (net 1))
   (via (at 144.907 98.298) (size 0.6) (drill 0.3) (layers F.Cu B.Cu) (net 1))
-  (via (at 141.097 97.536) (size 0.6) (drill 0.3) (layers F.Cu B.Cu) (net 1))
   (via (at 140.208 96.393) (size 0.6) (drill 0.3) (layers F.Cu B.Cu) (net 1))
   (via (at 139.7 94.996) (size 0.6) (drill 0.3) (layers F.Cu B.Cu) (net 1))
@@
   (via (at 128.143 120.015) (size 0.6) (drill 0.3) (layers F.Cu B.Cu) (net 1))
   (via (at 131.445 120.142) (size 0.6) (drill 0.3) (layers F.Cu B.Cu) (net 1))
-  (via (at 136.271 118.618) (size 0.6) (drill 0.3) (layers F.Cu B.Cu) (net 1))
+  (via (at 134.4676 119.38) (size 0.6) (drill 0.3) (layers F.Cu B.Cu) (net 1))
   (via (at 138.811 114.935) (size 0.6) (drill 0.3) (layers F.Cu B.Cu) (net 1))
   (via (at 140.589 113.03) (size 0.6) (drill 0.3) (layers F.Cu B.Cu) (net 1))
@@
   (via (at 115.062 102.108) (size 0.6) (drill 0.3) (layers F.Cu B.Cu) (net 1))
   (via (at 141.351 89.916) (size 0.6) (drill 0.3) (layers F.Cu B.Cu) (net 1))
-  (via (at 143.51 91.313) (size 0.6) (drill 0.3) (layers F.Cu B.Cu) (net 1))
+  (via (at 144.78 96.4692) (size 0.6) (drill 0.3) (layers F.Cu B.Cu) (net 1))
   (via (at 146.431 91.44) (size 0.6) (drill 0.3) (layers F.Cu B.Cu) (net 1))
-  (via (at 145.034 92.202) (size 0.6) (drill 0.3) (layers F.Cu B.Cu) (net 1))
+  (via (at 143.51 91.3384) (size 0.6) (drill 0.3) (layers F.Cu B.Cu) (net 1))
   (via (at 51.943 105.791) (size 0.6) (drill 0.3) (layers F.Cu B.Cu) (net 1))
   (via (at 51.562 118.745) (size 0.6) (drill 0.3) (layers F.Cu B.Cu) (net 1))
@@
   (via (at 70.358 85.598) (size 0.6) (drill 0.3) (layers F.Cu B.Cu) (net 1))
   (segment (start 69.701 89.938) (end 69.701 87.297) (width 0.6) (layer F.Cu) (net 1))
-  (via (at 69.701 89.938) (size 0.6) (drill 0.3) (layers F.Cu B.Cu) (net 1))
   (segment (start 69.70425 87.29375) (end 71.4 85.598) (width 0.6) (layer F.Cu) (net 1))
   (via (at 69.70425 87.29375) (size 0.6) (drill 0.3) (layers F.Cu B.Cu) (net 1))

Commit message: minor chages
Parts:
- added C51: 10u, Capacitor_Tantalum_SMD:CP_EIA-3216-18_Kemet-A, F.Cu at (140.0, 121.4)
- added C69: 10u, Capacitor_Tantalum_SMD:CP_EIA-3216-18_Kemet-A, F.Cu at (130.6, 50.0)
Connections:
- J2 pad 4: (no net) -> Net-(J2-Pad4)
- J2 pad 5: (no net) -> Net-(J2-Pad5)
- U1 pad 6: (no net) -> Net-(U1-Pad6)
- U1 pad 7: (no net) -> Net-(U1-Pad7)
- U13 pad 11: (no net) -> Net-(U13-Pad11)
- U13 pad 12: (no net) -> Net-(U13-Pad12)
- U13 pad 13: (no net) -> Net-(U13-Pad13)
- U13 pad 14: (no net) -> Net-(U13-Pad14)
- U13 pad 15: (no net) -> Net-(U13-Pad15)
- U13 pad 16: (no net) -> Net-(U13-Pad16)
- U13 pad 23: (no net) -> Net-(U13-Pad23)
- U13 pad 24: (no net) -> Net-(U13-Pad24)
- U13 pad 32: (no net) -> Net-(U13-Pad32)
- U13 pad 37: (no net) -> Net-(U13-Pad37)
- U13 pad 38: (no net) -> Net-(U13-Pad38)
- U13 pad 39: (no net) -> Net-(U13-Pad39)
- U13 pad 40: (no net) -> Net-(U13-Pad40)
- U13 pad 41: (no net) -> Net-(U13-Pad41)
- U13 pad 42: (no net) -> Net-(U13-Pad42)
- U13 pad 43: (no net) -> Net-(U13-Pad43)
- U13 pad 44: (no net) -> Net-(U13-Pad44)
- U13 pad 49: (no net) -> Net-(U13-Pad49)
- U13 pad 50: (no net) -> Net-(U13-Pad50)
- U13 pad 51: (no net) -> Net-(U13-Pad51)
- U13 pad 55: (no net) -> Net-(U13-Pad55)
- U13 pad 6: (no net) -> Net-(U13-Pad6)
- U13 pad 60: (no net) -> Net-(U13-Pad60)
- U13 pad 61: (no net) -> Net-(U13-Pad61)
- U13 pad 62: (no net) -> Net-(U13-Pad62)
- U13 pad 63: (no net) -> Net-(U13-Pad63)
- U13 pad 64: (no net) -> Net-(U13-Pad64)
- U13 pad 9: (no net) -> Net-(U13-Pad9)
- U6 pad 4: (no net) -> Net-(U6-Pad4)
- U7 pad 4: (no net) -> Net-(U7-Pad4)
- U8 pad 18: (no net) -> Net-(U8-Pad18)
- U8 pad 25: (no net) -> Net-(U8-Pad25)
Routing:
- net GND: track 105.9 -> 104.9 mm, vias 593 -> 596
- net VS_POS: vias 4 -> 5
- net +3V3: vias 9 -> 11

Commit message: first revision finished
Parts:
- added L3: Ferrite Bead, Capacitor_SMD:C_0603_1608Metric, F.Cu at (93.5, 135.4)
- added SW2: Button A, Button_Switch_THT:SW_Tactile_SPST_Angled_PTS645Vx58-2LFS, F.Cu at (144.0, 63.0)
- added SW3: Button B, Button_Switch_THT:SW_Tactile_SPST_Angled_PTS645Vx58-2LFS, F.Cu at (144.0, 73.4)
- added SW4: The Button, Button_Switch_THT:SW_Tactile_SPST_Angled_PTS645Vx58-2LFS, F.Cu at (144.0, 45.0)
- SW1: value PEC09-2120K -> EC11B152420G; footprint Potentiometers:Potentiometer_Alps_RK097_Double_Vertical -> kamtar:Potentiometer_Alps_RK097_Dual_Horizontal
- TP1: footprint Connect:1pin -> TestPoint:TestPoint_Plated_Hole_D2.0mm
- moved R29 11.0 mm to (124.7, 58.7), turned to 180 degrees
- moved R28 6.11 mm to (130.6, 55.4), turned to 270 degrees
- moved C57 5.59 mm to (135.1, 59.7), turned to 270 degrees
- moved R30 5.03 mm to (131.3, 62.0)
- moved C56 5.00 mm to (132.3, 55.4), turned to 270 degrees
- moved C58 3.56 mm to (133.0, 62.0)
- moved C69 1.98 mm to (129.0, 51.3), turned to 0 degrees
Connections:
- C24 pad 1: +3V3 -> /DykoDAC_CS4398/3V3_CS
- C25 pad 1: +3V3 -> /DykoDAC_CS4398/3V3_CS
- C26 pad 1: +3V3 -> /DykoDAC_CS4398/3V3_CS
- C27 pad 1: +3V3 -> /DykoDAC_CS4398/3V3_CS
- C56 pad 2: Net-(C56-Pad2) -> /DykoDAC_MCU/BA
- C57 pad 1: Net-(C57-Pad1) -> /DykoDAC_MCU/BB
- C69 pad 1: +3V3 -> /DykoDAC_MCU/3V3_Conn
- J8 pad 2: Net-(C56-Pad2) -> /DykoDAC_MCU/BA
- J8 pad 3: Net-(C57-Pad1) -> /DykoDAC_MCU/BB
- R28 pad 2: Net-(C56-Pad2) -> /DykoDAC_MCU/BA
- R29 pad 1: Net-(C57-Pad1) -> /DykoDAC_MCU/BB
- U8 pad 14: +3V3 -> /DykoDAC_CS4398/3V3_CS
- U8 pad 27: +3V3 -> /DykoDAC_CS4398/3V3_CS
- U8 pad 7: +3V3 -> /DykoDAC_CS4398/3V3_CS
Routing:
- net /DykoDAC_MCU/BB: track 0.00 -> 39.5 mm, vias 0 -> 1
- net +3V3: track 169.8 -> 137.7 mm, vias 11 -> 5
- net /DykoDAC_CS4398/3V3_CS: track 0.00 -> 30.5 mm, vias 0 -> 6
- net /DykoDAC_MCU/3V3_Conn: track 0.00 -> 28.0 mm
- net /DykoDAC_MCU/BTT: track 0.00 -> 27.9 mm, vias 0 -> 1
- net /DykoDAC_MCU/BA: track 0.00 -> 21.9 mm
- net GND: vias 596 -> 703
- added copper zone on F.Cu, net /DykoDAC_MCU/3V3_Conn
Other:
- board size 99.4 x 100.1 mm -> 99.2 x 99.8 mm
- board text added: "+5V"
- board text added: "+9V"
- board text added: "-9V"
- board text added: "AC 15V 1A"
- board text added: "CS4398 + TPA6120"
- board text added: "DIO"
- board text added: "GND"
- board text added: "Kamtar 2019"
- board text added: "OK"
- board text added: "RST"
- board text added: "RX"
- board text added: "TX"
- board text added: "V+ / Right"
- board text added: "V- / Left"
- board text added: "VS+"
- board text added: "VS-"
- board text removed: "15V 1A AC"
- board text removed: "AudioJack"
- board text removed: "POWER JACK"
- board text removed: "USB B"
