File: schematics/DykoDAC_Power.sch (KiCad schematic (older format))
At the start: 33 parts, among them J1 AC Input, U1 L7809, U2 L7909, U3 LT1762-5, U4 L7805, U5 LP5907-3.3

Commit message: finishing
Parts:
- C1: renamed from C9; footprint (none) -> Capacitors_SMD:C_1206
- C10: renamed from C7; footprint (none) -> Capacitors_SMD:C_1206
- C11: renamed from C8; footprint (none) -> Capacitors_SMD:C_1206
- C12: renamed from C11; footprint (none) -> Capacitors_SMD:C_1206
- C13, C16, C19, C21: renamed from C?; footprint (none) -> Capacitors_SMD:C_1206
- C14: renamed from C13; footprint (none) -> Capacitors_SMD:CP_Elec_8x6.7
- C15: renamed from C?; footprint (none) -> Capacitors_SMD:CP_Elec_8x6.7
- C17: renamed from C14; footprint (none) -> Capacitors_SMD:C_1206
- C18: renamed from C15; footprint (none) -> Capacitors_SMD:C_1206
- C2: renamed from C1; footprint (none) -> Capacitors_ThroughHole:CP_Radial_D5.0mm_P2.50mm
- C20: renamed from C16; footprint (none) -> Capacitors_SMD:C_1206
- C3: renamed from C2; footprint (none) -> Capacitors_ThroughHole:CP_Radial_D5.0mm_P2.50mm
- C4: renamed from C3; footprint (none) -> Capacitors_SMD:C_1206
- C5: renamed from C4; footprint (none) -> Capacitors_SMD:C_1206
- C6: renamed from C10; footprint (none) -> Capacitors_SMD:C_1206
- C7: renamed from C5; footprint (none) -> Capacitors_SMD:CP_Elec_8x6.7
- C8: renamed from C6; footprint (none) -> Capacitors_SMD:CP_Elec_8x6.7
- C9: renamed from C12; footprint (none) -> Capacitors_SMD:C_1206
- D1, D2: footprint (none) -> Capacitors_SMD:C_1206
- F1: renamed from F?; footprint (none) -> Fuse_Holders_and_Fuses:Fuse_SMD2920
- J1: footprint (none) -> Connect:BARREL_JACK
- L1: renamed from L?; footprint (none) -> Choke_SMD:Choke_SMD_1206_Standard
- U2: renamed from U1; footprint (none) -> TO_SOT_Packages_SMD:TO-263-2
- U3: renamed from U2; footprint (none) -> TO_SOT_Packages_SMD:TO-263-2
- U4: footprint (none) -> TO_SOT_Packages_SMD:TO-263-2
- U5: renamed from U?; footprint (none) -> TO_SOT_Packages_SMD:SOT-89-3
- gave numbers to parts that had none: 1
- renumbered U3 to U1, U5 to U6

Commit message: changed filter values started with PCB design
Parts:
- C19: value 1u -> 22u
- U6, U7: footprint Package_TO_SOT_SMD:SOT-23-5 -> TO_SOT_Packages_SMD:SOT-23-5
Other:
- moved on the sheet: C1, C6, C9, U1
Changed lines of the file:
@@
 L Regulator_Linear:LT1762-5 U1
 U 1 1 5C8D4B65
-P 3100 4600
-F 0 "U1" H 3100 5067 50  0000 C CNN
-F 1 "LT1762-5" H 3100 4976 50  0000 C CNN
-F 2 "Package_SO:MSOP-8_3x3mm_P0.65mm" H 3100 4250 50  0001 C CNN
-F 3 "https://www.analog.com/media/en/technical-documentation/data-sheets/LT1762.pdf" H 3100 4050 50  0001 C CNN
-	1    3100 4600
-	1    0    0    -1
-$EndComp
-Wire Wire Line
-	2700 4400 2550 4400
-Wire Wire Line
-	2150 4400 2150 4300
-Wire Wire Line
-	2700 4700 2550 4700
-Wire Wire Line
-	2550 4700 2550 4400
-Connection ~ 2550 4400
-Wire Wire Line
-	2550 4400 2150 4400
+P 3500 4600
+F 0 "U1" H 3500 5067 50  0000 C CNN
+F 1 "LT1762-5" H 3500 4976 50  0000 C CNN
+F 2 "Package_SO:MSOP-8_3x3mm_P0.65mm" H 3500 4250 50  0001 C CNN
+F 3 "https://www.analog.com/media/en/technical-documentation/data-sheets/LT1762.pdf" H 3500 4050 50  0001 C CNN
+	1    3500 4600
+	1    0    0    -1
+$EndComp
+Wire Wire Line
+	3100 4400 2950 4400
+Wire Wire Line
+	2550 4400 2550 4300
+Wire Wire Line
+	3100 4700 2950 4700
+Wire Wire Line
+	2950 4700 2950 4400
+Connection ~ 2950 4400
+Wire Wire Line
+	2950 4400 2550 4400
 $Comp
 L Device:C C1
 U 1 1 5C8D64CC
-P 2150 4650
-F 0 "C1" H 2265 4696 50  0000 L CNN
-F 1 "1u" H 2265 4605 50  0000 L CNN
-F 2 "Capacitors_SMD:C_1206" H 2188 4500 50  0001 C CNN
-F 3 "~" H 2150 4650 50  0001 C CNN
-	1    2150 4650
+P 2550 4650
+F 0 "C1" H 2665 4696 50  0000 L CNN
+F 1 "1u" H 2665 4605 50  0000 L CNN
+F 2 "Capacitors_SMD:C_1206" H 2588 4500 50  0001 C CNN
+F 3 "~" H 2550 4650 50  0001 C CNN
+	1    2550 4650
 	1    0    0    -1
 $EndComp
@@
 L power:GND #PWR03
 U 1 1 5C8D6589
-P 2150 5100
-F 0 "#PWR03" H 2150 4850 50  0001 C CNN
-F 1 "GND" H 2155 4927 50  0000 C CNN
-F 2 "" H 2150 5100 50  0001 C CNN
-F 3 "" H 2150 5100 50  0001 C CNN
-	1    2150 5100
-	1    0    0    -1
-$EndComp
-Wire Wire Line
-	2150 4500 2150 4400
-Connection ~ 2150 4400
-Wire Wire Line
-	2150 4800 2150 5000
-Wire Wire Line
-	3100 4900 3100 5000
-Wire Wire Line
-	3100 5000 2150 5000
-Connection ~ 2150 5000
-Wire Wire Line
-	2150 5000 2150 5100
+P 2550 5100
+F 0 "#PWR03" H 2550 4850 50  0001 C CNN
+F 1 "GND" H 2555 4927 50  0000 C CNN
+F 2 "" H 2550 5100 50  0001 C CNN
+F 3 "" H 2550 5100 50  0001 C CNN
+	1    2550 5100
+	1    0    0    -1
+$EndComp
+Wire Wire Line
+	2550 4500 2550 4400
+Connection ~ 2550 4400
+Wire Wire Line
+	2550 4800 2550 5000
+Wire Wire Line
+	3500 4900 3500 5000
+Wire Wire Line
+	3500 5000 2550 5000
+Connection ~ 2550 5000
+Wire Wire Line
+	2550 5000 2550 5100
 $Comp
 L power:+5VA #PWR05
 U 1 1 5C8D8B0E
-P 4300 4300
-F 0 "#PWR05" H 4300 4150 50  0001 C CNN
-F 1 "+5VA" H 4315 4473 50  0000 C CNN
-F 2 "" H 4300 4300 50  0001 C CNN
-F 3 "" H 4300 4300 50  0001 C CNN
-	1    4300 4300
-	1    0    0    -1
-$EndComp
-Wire Wire Line
-	3500 4400 3550 4400
-Wire Wire Line
-	4300 4400 4300 4300
+P 4700 4300
+F 0 "#PWR05" H 4700 4150 50  0001 C CNN
+F 1 "+5VA" H 4715 4473 50  0000 C CNN
+F 2 "" H 4700 4300 50  0001 C CNN
+F 3 "" H 4700 4300 50  0001 C CNN
+	1    4700 4300
+	1    0    0    -1
+$EndComp
+Wire Wire Line
+	3900 4400 3950 4400
+Wire Wire Line
+	4700 4400 4700 4300
 $Comp
 L Device:C C6
 U 1 1 5C8D9A44
-P 3800 4650
-F 0 "C6" H 3915 4696 50  0000 L CNN
-F 1 "10n" H 3915 4605 50  0000 L CNN
-F 2 "Capacitors_SMD:C_1206" H 3838 4500 50  0001 C CNN
-F 3 "~" H 3800 4650 50  0001 C CNN
-	1    3800 4650
-	1    0    0    -1
-$EndComp
-Wire Wire Line
-	3500 4700 3600 4700
-Wire Wire Line
-	3600 4700 3600 4850
-Wire Wire Line
-	3600 4850 3800 4850
-Wire Wire Line
-	3800 4850 3800 4800
-Wire Wire Line
-	3800 4500 3550 4500
-Wire Wire Line
-	3550 4500 3550 4400
-Connection ~ 3550 4500
-Wire Wire Line
-	3550 4500 3500 4500
-Connection ~ 3550 4400
-Wire Wire Line
-	3550 4400 4300 4400
+P 4200 4650
+F 0 "C6" H 4315 4696 50  0000 L CNN
+F 1 "10n" H 4315 4605 50  0000 L CNN
+F 2 "Capacitors_SMD:C_1206" H 4238 4500 50  0001 C CNN
+F 3 "~" H 4200 4650 50  0001 C CNN
+	1    4200 4650
+	1    0    0    -1
+$EndComp
+Wire Wire Line
+	3900 4700 4000 4700
+Wire Wire Line
+	4000 4700 4000 4850
+Wire Wire Line
+	4000 4850 4200 4850
+Wire Wire Line
+	4200 4850 4200 4800
+Wire Wire Line
+	4200 4500 3950 4500
+Wire Wire Line
+	3950 4500 3950 4400
+Connection ~ 3950 4500
+Wire Wire Line
+	3950 4500 3900 4500
+Connection ~ 3950 4400
+Wire Wire Line
+	3950 4400 4700 4400
 $Comp
 L Device:CP C9
 U 1 1 5C8DCF89
-P 4300 4650
-F 0 "C9" H 4418 4696 50  0000 L CNN
-F 1 "10u" H 4418 4605 50  0000 L CNN
-F 2 "Capacitors_SMD:C_1206" H 4338 4500 50  0001 C CNN
-F 3 "~" H 4300 4650 50  0001 C CNN
-	1    4300 4650
-	1    0    0    -1
-$EndComp
-Wire Wire Line
-	4300 4500 4300 4400
-Connection ~ 4300 4400
-Wire Wire Line
-	4300 4800 4300 5000
-Wire Wire Line
-	4300 5000 3100 5000
-Connection ~ 3100 5000
+P 4700 4650
+F 0 "C9" H 4818 4696 50  0000 L CNN
+F 1 "10u" H 4818 4605 50  0000 L CNN
+F 2 "Capacitors_SMD:C_1206" H 4738 4500 50  0001 C CNN
+F 3 "~" H 4700 4650 50  0001 C CNN
+	1    4700 4650
+	1    0    0    -1
+$EndComp
+Wire Wire Line
+	4700 4500 4700 4400
+Connection ~ 4700 4400
+Wire Wire Line
+	4700 4800 4700 5000
+Wire Wire Line
+	4700 5000 3500 5000
+Connection ~ 3500 5000
 $Comp
 L Regulator_Linear:LP5907MFX-1.8 U6
@@
 F 0 "U6" H 8950 2567 50  0000 C CNN
 F 1 "LP5907-3.3" H 8950 2476 50  0000 C CNN
-F 2 "Package_TO_SOT_SMD:SOT-23-5" H 8950 2550 50  0001 C CNN
+F 2 "TO_SOT_Packages_SMD:SOT-23-5" H 8950 2550 50  0001 C CNN
 F 3 "http://www.ti.com/lit/ds/symlink/lp5907.pdf" H 8950 2700 50  0001 C CNN
 	1    8950 2200
@@
 Text Notes 8850 1600 0    118  ~ 0
 Digital
-Text Notes 3700 4000 0    118  ~ 0
+Text Notes 4100 4000 0    118  ~ 0
 DAC Analog
 $Comp
 L power:+9V #PWR02
 U 1 1 5C8C6769
-P 2150 4300
-F 0 "#PWR02" H 2150 4150 50  0001 C CNN
-F 1 "+9V" H 2165 4473 50  0000 C CNN
-F 2 "" H 2150 4300 50  0001 C CNN
-F 3 "" H 2150 4300 50  0001 C CNN
-	1    2150 4300
+P 2550 4300
+F 0 "#PWR02" H 2550 4150 50  0001 C CNN
+F 1 "+9V" H 2565 4473 50  0000 C CNN
+F 2 "" H 2550 4300 50  0001 C CNN
+F 3 "" H 2550 4300 50  0001 C CNN
+	1    2550 4300
 	1    0    0    -1
 $EndComp
@@
 F 0 "U7" H 8950 4867 50  0000 C CNN
 F 1 "LP5907-3.3" H 8950 4776 50  0000 C CNN
-F 2 "Package_TO_SOT_SMD:SOT-23-5" H 8950 4850 50  0001 C CNN
+F 2 "TO_SOT_Packages_SMD:SOT-23-5" H 8950 4850 50  0001 C CNN
 F 3 "http://www.ti.com/lit/ds/symlink/lp5907.pdf" H 8950 5000 50  0001 C CNN
 	1    8950 4500
@@
 P 8400 4650
 F 0 "C19" H 8515 4696 50  0000 L CNN
-F 1 "1u" H 8515 4605 50  0000 L CNN
+F 1 "22u" H 8515 4605 50  0000 L CNN
 F 2 "Capacitors_SMD:C_1206" H 8438 4500 50  0001 C CNN
 F 3 "~" H 8400 4650 50  0001 C CNN

Commit message: pcb dev.
Parts:
- C2, C3: footprint Capacitors_ThroughHole:CP_Radial_D5.0mm_P2.50mm -> kamtar:CP_Radial_D16.0mm_P7.50mm_Hor
Changed lines of the file:
@@
 F 0 "C2" H 2868 2046 50  0000 L CNN
 F 1 "4700u" H 2868 1955 50  0000 L CNN
-F 2 "Capacitors_ThroughHole:CP_Radial_D5.0mm_P2.50mm" H 2788 1850 50  0001 C CNN
+F 2 "kamtar:CP_Radial_D16.0mm_P7.50mm_Hor" H 2788 1850 50  0001 C CNN
 F 3 "~" H 2750 2000 50  0001 C CNN
 	1    2750 2000
@@
 F 0 "C3" H 2868 2546 50  0000 L CNN
 F 1 "4700u" H 2868 2455 50  0000 L CNN
-F 2 "Capacitors_ThroughHole:CP_Radial_D5.0mm_P2.50mm" H 2788 2350 50  0001 C CNN
+F 2 "kamtar:CP_Radial_D16.0mm_P7.50mm_Hor" H 2788 2350 50  0001 C CNN
 F 3 "~" H 2750 2500 50  0001 C CNN
 	1    2750 2500

Commit message: lots of stuf ....
Parts:
- C1, C10, C11, C12, C13, C16, C17, C18, C19, C20, C21, C4, C5, C6, C9: footprint Capacitors_SMD:C_1206 -> Capacitors_SMD:C_0603_HandSoldering
- D1, D2: footprint Capacitors_SMD:C_1206 -> Diodes_SMD:D_SMB_Handsoldering
- U1: footprint Package_SO:MSOP-8_3x3mm_P0.65mm -> Housings_SSOP:MSOP-8_3x3mm_Pitch0.65mm
Changed lines of the file:
@@
 F 0 "D1" V 2154 2079 50  0000 L CNN
 F 1 "D" V 2245 2079 50  0000 L CNN
-F 2 "Capacitors_SMD:C_1206" H 2200 2000 50  0001 C CNN
+F 2 "Diodes_SMD:D_SMB_Handsoldering" H 2200 2000 50  0001 C CNN
 F 3 "~" H 2200 2000 50  0001 C CNN
 	1    2200 2000
@@
 F 0 "D2" V 2154 2579 50  0000 L CNN
 F 1 "D" V 2245 2579 50  0000 L CNN
-F 2 "Capacitors_SMD:C_1206" H 2200 2500 50  0001 C CNN
+F 2 "Diodes_SMD:D_SMB_Handsoldering" H 2200 2500 50  0001 C CNN
 F 3 "~" H 2200 2500 50  0001 C CNN
 	1    2200 2500
@@
 F 0 "C10" H 4815 1996 50  0000 L CNN
 F 1 "100n" H 4815 1905 50  0000 L CNN
-F 2 "Capacitors_SMD:C_1206" H 4738 1800 50  0001 C CNN
+F 2 "Capacitors_SMD:C_0603_HandSoldering" H 4738 1800 50  0001 C CNN
 F 3 "~" H 4700 1950 50  0001 C CNN
 	1    4700 1950
@@
 F 0 "C11" H 4815 2546 50  0000 L CNN
 F 1 "100n" H 4815 2455 50  0000 L CNN
-F 2 "Capacitors_SMD:C_1206" H 4738 2350 50  0001 C CNN
+F 2 "Capacitors_SMD:C_0603_HandSoldering" H 4738 2350 50  0001 C CNN
 F 3 "~" H 4700 2500 50  0001 C CNN
 	1    4700 2500
@@
 F 0 "C4" H 3565 2046 50  0000 L CNN
 F 1 "100n" H 3565 1955 50  0000 L CNN
-F 2 "Capacitors_SMD:C_1206" H 3488 1850 50  0001 C CNN
+F 2 "Capacitors_SMD:C_0603_HandSoldering" H 3488 1850 50  0001 C CNN
 F 3 "~" H 3450 2000 50  0001 C CNN
 	1    3450 2000
@@
 F 0 "C5" H 3350 2650 50  0000 R CNN
 F 1 "100n" H 3350 2550 50  0000 R CNN
-F 2 "Capacitors_SMD:C_1206" H 3488 2350 50  0001 C CNN
+F 2 "Capacitors_SMD:C_0603_HandSoldering" H 3488 2350 50  0001 C CNN
 F 3 "~" H 3450 2500 50  0001 C CNN
 	1    3450 2500
@@
 F 0 "U1" H 3500 5067 50  0000 C CNN
 F 1 "LT1762-5" H 3500 4976 50  0000 C CNN
-F 2 "Package_SO:MSOP-8_3x3mm_P0.65mm" H 3500 4250 50  0001 C CNN
+F 2 "Housings_SSOP:MSOP-8_3x3mm_Pitch0.65mm" H 3500 4250 50  0001 C CNN
 F 3 "https://www.analog.com/media/en/technical-documentation/data-sheets/LT1762.pdf" H 3500 4050 50  0001 C CNN
 	1    3500 4600
@@
 F 0 "C1" H 2665 4696 50  0000 L CNN
 F 1 "1u" H 2665 4605 50  0000 L CNN
-F 2 "Capacitors_SMD:C_1206" H 2588 4500 50  0001 C CNN
+F 2 "Capacitors_SMD:C_0603_HandSoldering" H 2588 4500 50  0001 C CNN
 F 3 "~" H 2550 4650 50  0001 C CNN
 	1    2550 4650
@@
 F 0 "C6" H 4315 4696 50  0000 L CNN
 F 1 "10n" H 4315 4605 50  0000 L CNN
-F 2 "Capacitors_SMD:C_1206" H 4238 4500 50  0001 C CNN
+F 2 "Capacitors_SMD:C_0603_HandSoldering" H 4238 4500 50  0001 C CNN
 F 3 "~" H 4200 4650 50  0001 C CNN
 	1    4200 4650
@@
 F 0 "C9" H 4818 4696 50  0000 L CNN
 F 1 "10u" H 4818 4605 50  0000 L CNN
-F 2 "Capacitors_SMD:C_1206" H 4738 4500 50  0001 C CNN
+F 2 "Capacitors_SMD:C_0603_HandSoldering" H 4738 4500 50  0001 C CNN
 F 3 "~" H 4700 4650 50  0001 C CNN
 	1    4700 4650
@@
 F 0 "C18" H 8515 2396 50  0000 L CNN
 F 1 "1u" H 8515 2305 50  0000 L CNN
-F 2 "Capacitors_SMD:C_1206" H 8438 2200 50  0001 C CNN
+F 2 "Capacitors_SMD:C_0603_HandSoldering" H 8438 2200 50  0001 C CNN
 F 3 "~" H 8400 2350 50  0001 C CNN
 	1    8400 2350
@@
 F 0 "C17" H 8065 2396 50  0000 L CNN
 F 1 "100n" H 8065 2305 50  0000 L CNN
-F 2 "Capacitors_SMD:C_1206" H 7988 2200 50  0001 C CNN
+F 2 "Capacitors_SMD:C_0603_HandSoldering" H 7988 2200 50  0001 C CNN
 F 3 "~" H 7950 2350 50  0001 C CNN
 	1    7950 2350
@@
 F 0 "C12" H 6715 2396 50  0000 L CNN
 F 1 "100n" H 6715 2305 50  0000 L CNN
-F 2 "Capacitors_SMD:C_1206" H 6638 2200 50  0001 C CNN
+F 2 "Capacitors_SMD:C_0603_HandSoldering" H 6638 2200 50  0001 C CNN
 F 3 "~" H 6600 2350 50  0001 C CNN
 	1    6600 2350
@@
 F 0 "C20" H 9515 2396 50  0000 L CNN
 F 1 "1u" H 9515 2305 50  0000 L CNN
-F 2 "Capacitors_SMD:C_1206" H 9438 2200 50  0001 C CNN
+F 2 "Capacitors_SMD:C_0603_HandSoldering" H 9438 2200 50  0001 C CNN
 F 3 "~" H 9400 2350 50  0001 C CNN
 	1    9400 2350
@@
 F 0 "C19" H 8515 4696 50  0000 L CNN
 F 1 "22u" H 8515 4605 50  0000 L CNN
-F 2 "Capacitors_SMD:C_1206" H 8438 4500 50  0001 C CNN
+F 2 "Capacitors_SMD:C_0603_HandSoldering" H 8438 4500 50  0001 C CNN
 F 3 "~" H 8400 4650 50  0001 C CNN
 	1    8400 4650
@@
 F 0 "C16" H 7915 4696 50  0000 L CNN
 F 1 "100n" H 7915 4605 50  0000 L CNN
-F 2 "Capacitors_SMD:C_1206" H 7838 4500 50  0001 C CNN
+F 2 "Capacitors_SMD:C_0603_HandSoldering" H 7838 4500 50  0001 C CNN
 F 3 "~" H 7800 4650 50  0001 C CNN
 	1    7800 4650
@@
 F 0 "C13" H 6715 4696 50  0000 L CNN
 F 1 "100n" H 6715 4605 50  0000 L CNN
-F 2 "Capacitors_SMD:C_1206" H 6638 4500 50  0001 C CNN
+F 2 "Capacitors_SMD:C_0603_HandSoldering" H 6638 4500 50  0001 C CNN
 F 3 "~" H 6600 4650 50  0001 C CNN
 	1    6600 4650
@@
 F 0 "C21" H 9515 4696 50  0000 L CNN
 F 1 "1u" H 9515 4605 50  0000 L CNN
-F 2 "Capacitors_SMD:C_1206" H 9438 4500 50  0001 C CNN
+F 2 "Capacitors_SMD:C_0603_HandSoldering" H 9438 4500 50  0001 C CNN
 F 3 "~" H 9400 4650 50  0001 C CNN
 	1    9400 4650

Commit message: no message
Parts:
- removed U2: L7809, TO_SOT_Packages_SMD:TO-263-2, symbol Regulator_Linear:L7809
- removed U3: L7909, TO_SOT_Packages_SMD:TO-263-2, symbol Regulator_Linear:LM7909_TO220
- added C64, C65: 10u, symbol Device:CP_Small
- added R40, R43: 240, symbol Device:R_Small
- added R41, R42: 1k5, symbol Device:R_Small
- added U2: LM317, TO_SOT_Packages_SMD:TO-263-2, symbol Regulator_Linear:LM337_SOT223
- added U3: LM337, TO_SOT_Packages_SMD:TO-263-2, symbol Regulator_Linear:LM337_SOT223
- C1, C10, C11, C12, C16, C17, C18, C19, C20, C21, C4, C5, C6: footprint Capacitors_SMD:C_0603_HandSoldering -> Capacitors_SMD:C_0603
- C9: footprint Capacitors_SMD:C_0603_HandSoldering -> Capacitors_SMD:CP_Elec_4x5.7
- D1, D2: footprint Diodes_SMD:D_SMB_Handsoldering -> Diodes_SMD:D_SMB
- L1: value 100u -> Ferrite Bead; footprint Choke_SMD:Choke_SMD_1206_Standard -> Capacitors_SMD:C_0603
Connections:
- wire segments 134 -> 151
Other:
- note removed: "Op-Amp Power"
- moved on the sheet: C10, C11, C2, C3, C4, C5, C7, C8
