File: schematics/DykoDAC_Power.sch (KiCad schematic (older format))
At the start: 35 parts, among them J1 AC Input, SW5 PWR_SWITCH, U1 LT1762-5, U2 L7812, U3 L7912, U4 L7805, U5 78l05, U6 LP5907-3.3, U7 LP5907-3.3

Commit message: minor changes & pdf update
Other:
- note added: "Designed for 15V/1A transformer"
- moved on the sheet: C1, C10, C11, C14, C15, C16, C17, C2, C3, C4, C5, C6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

Commit message: cosmetic changes
Parts:
- C10, C11, C12, C13, C16, C17, C4, C5: value 100n -> 0.1u
Changed lines of the file:
@@
 P 4550 1850
 F 0 "C10" H 4665 1896 50  0000 L CNN
-F 1 "100n" H 4665 1805 50  0000 L CNN
+F 1 "0.1u" H 4665 1805 50  0000 L CNN
 F 2 "Capacitors_SMD:C_0603" H 4588 1700 50  0001 C CNN
 F 3 "~" H 4550 1850 50  0001 C CNN
@@
 P 4550 2550
 F 0 "C11" H 4665 2596 50  0000 L CNN
-F 1 "100n" H 4665 2505 50  0000 L CNN
+F 1 "0.1u" H 4665 2505 50  0000 L CNN
 F 2 "Capacitors_SMD:C_0603" H 4588 2400 50  0001 C CNN
 F 3 "~" H 4550 2550 50  0001 C CNN
@@
 P 3650 1850
 F 0 "C4" H 3765 1896 50  0000 L CNN
-F 1 "100n" H 3765 1805 50  0000 L CNN
+F 1 "0.1u" H 3765 1805 50  0000 L CNN
 F 2 "Capacitors_SMD:C_0603" H 3688 1700 50  0001 C CNN
 F 3 "~" H 3650 1850 50  0001 C CNN
@@
 P 3650 2650
 F 0 "C5" H 3550 2800 50  0000 R CNN
-F 1 "100n" H 3550 2700 50  0000 R CNN
+F 1 "0.1u" H 3550 2700 50  0000 R CNN
 F 2 "Capacitors_SMD:C_0603" H 3688 2500 50  0001 C CNN
 F 3 "~" H 3650 2650 50  0001 C CNN
@@
 P 7550 2350
 F 0 "C17" H 7300 2350 50  0000 L CNN
-F 1 "100n" H 7300 2250 50  0000 L CNN
+F 1 "0.1u" H 7300 2250 50  0000 L CNN
 F 2 "Capacitors_SMD:C_0603" H 7588 2200 50  0001 C CNN
 F 3 "~" H 7550 2350 50  0001 C CNN
@@
 P 6600 2350
 F 0 "C12" H 6715 2396 50  0000 L CNN
-F 1 "100n" H 6715 2305 50  0000 L CNN
+F 1 "0.1u" H 6715 2305 50  0000 L CNN
 F 2 "Capacitors_SMD:C_0603" H 6638 2200 50  0001 C CNN
 F 3 "~" H 6600 2350 50  0001 C CNN
@@
 P 7550 4650
 F 0 "C16" H 7300 4650 50  0000 L CNN
-F 1 "100n" H 7300 4550 50  0000 L CNN
+F 1 "0.1u" H 7300 4550 50  0000 L CNN
 F 2 "Capacitors_SMD:C_0603" H 7588 4500 50  0001 C CNN
 F 3 "~" H 7550 4650 50  0001 C CNN
@@
 P 6600 4650
 F 0 "C13" H 6715 4696 50  0000 L CNN
-F 1 "100n" H 6715 4605 50  0000 L CNN
+F 1 "0.1u" H 6715 4605 50  0000 L CNN
 F 2 "Capacitors_SMD:C_0603" H 6638 4500 50  0001 C CNN
 F 3 "~" H 6600 4650 50  0001 C CNN

Commit message: new pdf and minor changes in schematics and fw
Parts:
- U5: symbol kamtar:78l05 -> DykoDAC-rescue:78l05-kamtar
Changed lines of the file:
@@
 $EndComp
 $Comp
-L kamtar:78l05 U5
+L DykoDAC-rescue:78l05-kamtar U5
 U 1 1 5E735AE7
 P 7150 4400
+AR Path="/5E735AE7" Ref="U5"  Part="1"
+AR Path="/5C91BC19/5E735AE7" Ref="U5"  Part="1"
 F 0 "U5" H 7150 4642 50  0000 C CNN
 F 1 "78l05" H 7150 4551 50  0000 C CNN
