File: schematics/DykoDAC_CS4398.sch (KiCad schematic (older format))
At the start: 20 parts, among them U8 CS4398, X1 22.5792Mhz, X2 24.576Mhz

Commit message: no message
Parts:
- X2: Part (none) -> NDK NZ2520SD
Other:
- note added: "NDK NZ2520SD Crystal Oscillators"
Changed lines of the file:
@@
 F 2 "Oscillators:Oscillator_SMD_SeikoEpson_SG210-4pin_2.5x2.0mm_HandSoldering" H 3350 4350 50  0001 C CNN
 F 3 "http://www.txccorp.com/download/products/osc/7C_o.pdf" H 2550 4700 50  0001 C CNN
-F 4 "NDK NZ2520SD" H 3200 4850 50  0000 C CNN "Part"
+F 4 "NDK NZ2520SD" H 3300 4800 50  0001 C CNN "Part"
 	1    2650 4700
 	1    0    0    -1
@@
 F 2 "Oscillators:Oscillator_SMD_SeikoEpson_SG210-4pin_2.5x2.0mm_HandSoldering" H 3350 5900 50  0001 C CNN
 F 3 "http://www.txccorp.com/download/products/osc/7C_o.pdf" H 2550 6250 50  0001 C CNN
+F 4 "NDK NZ2520SD" H 2650 6250 50  0001 C CNN "Part"
 	1    2650 6250
 	1    0    0    -1
@@
 Wire Wire Line
 	5800 3550 7150 3550
+Text Notes 1250 3750 0    79   ~ 0
+NDK NZ2520SD Crystal Oscillators
 $EndSCHEMATC

Commit message: first revision finished
Parts:
- added L3: Ferrite Bead, Capacitor_SMD:C_0603_1608Metric, symbol Device:L
Connections:
- net +3V3: now also L3.1; no longer C24.1, C25.1, C26.1, C27.1, U8.14 (VLC), U8.27 (VLS), U8.7 (VD)
- new net 3V3_CS: C24.1, C25.1, C26.1, C27.1, L3.2, U8.14 (VLC), U8.27 (VLS), U8.7 (VD)
Changed lines of the file:
@@
 L power:+3.3V #PWR021
 U 1 1 5C8F8A9A
-P 7150 1950
-F 0 "#PWR021" H 7150 1800 50  0001 C CNN
-F 1 "+3.3V" V 7165 2078 50  0000 L CNN
-F 2 "" H 7150 1950 50  0001 C CNN
-F 3 "" H 7150 1950 50  0001 C CNN
-	1    7150 1950
+P 6550 1950
+F 0 "#PWR021" H 6550 1800 50  0001 C CNN
+F 1 "+3.3V" V 6565 2078 50  0000 L CNN
+F 2 "" H 6550 1950 50  0001 C CNN
+F 3 "" H 6550 1950 50  0001 C CNN
+	1    6550 1950
 	0    -1   -1   0
 $EndComp
@@
 Wire Wire Line
 	7400 1850 7400 1950
-Connection ~ 7400 1950
-Wire Wire Line
-	7400 1950 7150 1950
 Wire Wire Line
 	7750 1850 7750 1950
@@
 	1    0    0    -1
 $EndComp
-$Comp
-L power:+3.3V #PWR017
-U 1 1 5C901381
-P 6100 2950
-F 0 "#PWR017" H 6100 2800 50  0001 C CNN
-F 1 "+3.3V" V 6115 3078 50  0000 L CNN
-F 2 "" H 6100 2950 50  0001 C CNN
-F 3 "" H 6100 2950 50  0001 C CNN
-	1    6100 2950
-	0    -1   -1   0
-$EndComp
-$Comp
-L power:+3.3V #PWR015
-U 1 1 5C9013EB
-P 5700 3550
-F 0 "#PWR015" H 5700 3400 50  0001 C CNN
-F 1 "+3.3V" V 5715 3678 50  0000 L CNN
-F 2 "" H 5700 3550 50  0001 C CNN
-F 3 "" H 5700 3550 50  0001 C CNN
-	1    5700 3550
-	0    -1   -1   0
-$EndComp
-Wire Wire Line
-	6100 2950 6250 2950
 Wire Wire Line
 	6250 2850 6250 2950
@@
 Text Notes 1250 3750 0    79   ~ 0
 NDK NZ2520SD Crystal Oscillators
+$Comp
+L Device:L L?
+U 1 1 5E71E0D1
+P 6800 1950
+AR Path="/5C91BC19/5E71E0D1" Ref="L?"  Part="1"
+AR Path="/5C8F8588/5E71E0D1" Ref="L3"  Part="1"
+F 0 "L3" V 6990 1950 50  0000 C CNN
+F 1 "Ferrite Bead" V 6899 1950 50  0000 C CNN
+F 2 "Capacitor_SMD:C_0603_1608Metric" H 6800 1950 50  0001 C CNN
+F 3 "~" H 6800 1950 50  0001 C CNN
+	1    6800 1950
+	0    -1   -1   0
+$EndComp
+Connection ~ 7400 1950
+Text Label 7100 1650 0    47   ~ 0
+3V3_CS
+Wire Wire Line
+	6950 1950 7100 1950
+Wire Wire Line
+	6650 1950 6550 1950
+Wire Wire Line
+	7100 1650 7100 1950
+Connection ~ 7100 1950
+Wire Wire Line
+	7100 1950 7400 1950
+Text Label 5800 2950 0    47   ~ 0
+3V3_CS
+Wire Wire Line
+	5800 2950 6250 2950
+Text Label 5700 3550 0    47   ~ 0
+3V3_CS
 $EndSCHEMATC

Commit message: update
Parts:
- added C70: 10u, Capacitor_Tantalum_SMD:CP_EIA-3216-18_Kemet-A, symbol Device:CP
- C26, C29, C33: footprint Capacitors_Tantalum_SMD:CP_Tantalum_Case-A_EIA-3216-18_Reflow -> Capacitor_Tantalum_SMD:CP_EIA-3216-18_Kemet-A
- C32: footprint Capacitors_Tantalum_SMD:CP_Tantalum_Case-D_EIA-7343-31_Reflow -> Capacitor_Tantalum_SMD:CP_EIA-7343-31_Kemet-D
Connections:
- net +3V3: now also C70.1
- net GND: now also C70.2
Changed lines of the file:
@@
 F 0 "C26" H 7282 1654 50  0000 R CNN
 F 1 "10u" H 7282 1745 50  0000 R CNN
-F 2 "Capacitors_Tantalum_SMD:CP_Tantalum_Case-A_EIA-3216-18_Reflow" H 7438 1550 50  0001 C CNN
+F 2 "Capacitor_Tantalum_SMD:CP_EIA-3216-18_Kemet-A" H 7438 1550 50  0001 C CNN
 F 3 "~" H 7400 1700 50  0001 C CNN
 	1    7400 1700
@@
 F 0 "C29" H 8532 1654 50  0000 R CNN
 F 1 "10u" H 8532 1745 50  0000 R CNN
-F 2 "Capacitors_Tantalum_SMD:CP_Tantalum_Case-A_EIA-3216-18_Reflow" H 8688 1550 50  0001 C CNN
+F 2 "Capacitor_Tantalum_SMD:CP_EIA-3216-18_Kemet-A" H 8688 1550 50  0001 C CNN
 F 3 "~" H 8650 1700 50  0001 C CNN
 	1    8650 1700
@@
 L power:+3.3V #PWR021
 U 1 1 5C8F8A9A
-P 6550 1950
-F 0 "#PWR021" H 6550 1800 50  0001 C CNN
-F 1 "+3.3V" V 6565 2078 50  0000 L CNN
-F 2 "" H 6550 1950 50  0001 C CNN
-F 3 "" H 6550 1950 50  0001 C CNN
-	1    6550 1950
+P 6150 1950
+F 0 "#PWR021" H 6150 1800 50  0001 C CNN
+F 1 "+3.3V" V 6165 2078 50  0000 L CNN
+F 2 "" H 6150 1950 50  0001 C CNN
+F 3 "" H 6150 1950 50  0001 C CNN
+	1    6150 1950
 	0    -1   -1   0
 $EndComp
@@
 F 0 "C32" H 9800 3900 50  0000 L CNN
 F 1 "100u" H 9800 3700 50  0000 L CNN
-F 2 "Capacitors_Tantalum_SMD:CP_Tantalum_Case-D_EIA-7343-31_Reflow" H 9788 3650 50  0001 C CNN
+F 2 "Capacitor_Tantalum_SMD:CP_EIA-7343-31_Kemet-D" H 9788 3650 50  0001 C CNN
 F 3 "~" H 9750 3800 50  0001 C CNN
 F 4 "TAJD107K016SNJ" H 9750 3800 50  0001 C CNN "Part"
@@
 F 0 "C33" H 9632 4204 50  0000 R CNN
 F 1 "33u" H 9632 4295 50  0000 R CNN
-F 2 "Capacitors_Tantalum_SMD:CP_Tantalum_Case-A_EIA-3216-18_Reflow" H 9788 4100 50  0001 C CNN
+F 2 "Capacitor_Tantalum_SMD:CP_EIA-3216-18_Kemet-A" H 9788 4100 50  0001 C CNN
 F 3 "~" H 9750 4250 50  0001 C CNN
 	1    9750 4250
@@
 	6950 1950 7100 1950
 Wire Wire Line
-	6650 1950 6550 1950
-Wire Wire Line
 	7100 1650 7100 1950
 Connection ~ 7100 1950
@@
 Text Label 5700 3550 0    47   ~ 0
 3V3_CS
+Wire Wire Line
+	6150 1950 6300 1950
+$Comp
+L Device:CP C70
+U 1 1 5E6B16EE
+P 6300 1750
+F 0 "C70" H 6182 1704 50  0000 R CNN
+F 1 "10u" H 6182 1795 50  0000 R CNN
+F 2 "Capacitor_Tantalum_SMD:CP_EIA-3216-18_Kemet-A" H 6338 1600 50  0001 C CNN
+F 3 "~" H 6300 1750 50  0001 C CNN
+	1    6300 1750
+	-1   0    0    1
+$EndComp
+$Comp
+L power:GND #PWR015
+U 1 1 5E6B2E29
+P 6300 1500
+F 0 "#PWR015" H 6300 1250 50  0001 C CNN
+F 1 "GND" H 6305 1327 50  0000 C CNN
+F 2 "" H 6300 1500 50  0001 C CNN
+F 3 "" H 6300 1500 50  0001 C CNN
+	1    6300 1500
+	-1   0    0    1
+$EndComp
+Wire Wire Line
+	6300 1600 6300 1500
+Wire Wire Line
+	6300 1900 6300 1950
+Connection ~ 6300 1950
+Wire Wire Line
+	6300 1950 6650 1950
 $EndSCHEMATC

Commit message: cosmetic changes
Changed lines of the file:
@@
 U 1 1 5C8FFC64
 P 5800 3800
-F 0 "C24" H 5900 3850 50  0000 L CNN
-F 1 "0.1u" H 5915 3755 50  0000 L CNN
+F 0 "C24" H 5500 3850 50  0000 L CNN
+F 1 "0.1u" H 5500 3750 50  0000 L CNN
 F 2 "Capacitors_SMD:C_0603" H 5838 3650 50  0001 C CNN
 F 3 "~" H 5800 3800 50  0001 C CNN
@@
 U 1 1 5E6B16EE
 P 6300 1750
-F 0 "C70" H 6182 1704 50  0000 R CNN
-F 1 "10u" H 6182 1795 50  0000 R CNN
+F 0 "C70" H 6550 1700 50  0000 R CNN
+F 1 "10u" H 6550 1800 50  0000 R CNN
 F 2 "Capacitor_Tantalum_SMD:CP_EIA-3216-18_Kemet-A" H 6338 1600 50  0001 C CNN
 F 3 "~" H 6300 1750 50  0001 C CNN
